File: zikzak3/zikzak3-memswitch3.sch (EAGLE design)
At the start: 44 parts, among them IC2 MEGA128-A, Q1 16MHz, Q2 20MHz

Commit message: Some new code for cpu and gpu, clarified schematic
Connections:
- new net N$122: GPU.PCINT1/ADC1_PA1, X1-13.F
- new net N$124: GPU.PCINT2/ADC2_PA2, X1-14.F
- new net N$125: BUFFER3A.G, GPU.PCINT0/ADC0_PA0
- net GND: now also CONTROLA.G, MUX1A.G, MUX2A.G, MUX3A.G, MUX4A.G, MUX6A.G, MUX7A.G, MUX8A.G
- net N$119: now also X1-1.F; no longer X1-3.F
- net N$121: now also X1-2.F; no longer X1-8.F
- net N$123: now also X1-3.F; no longer X1-13.F
Other:
- note added: "Actually, swap these A<->B"
- note added: "Always A -> B"
- note added: "BB"
- note added: "GG"
- note added: "HSync"
- note added: "RR"
- note added: "VGA Blanker"
- note added: "VSync"
Changed lines of the file:
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@@
 <part name="INVERTOR" library="74xx-us" deviceset="74*04" device="N" technology="LS"/>
 <part name="BUFFER3" library="74xx-us" deviceset="74*245" device="N" technology="LS"/>
+<part name="P+7" library="supply1" deviceset="+5V" device=""/>
+<part name="GND8" library="supply1" deviceset="GND" device=""/>
+<part name="GND9" library="supply1" deviceset="GND" device=""/>
+<part name="GND15" library="supply1" deviceset="GND" device=""/>
+<part name="GND16" library="supply1" deviceset="GND" device=""/>
+<part name="GND17" library="supply1" deviceset="GND" device=""/>
+<part name="GND18" library="supply1" deviceset="GND" device=""/>
+<part name="GND19" library="supply1" deviceset="GND" device=""/>
+<part name="GND20" library="supply1" deviceset="GND" device=""/>
+<part name="GND21" library="supply1" deviceset="GND" device=""/>
 </parts>
 <sheets>
@@
 <text x="-111.76" y="53.34" size="6.4516" layer="91">JOY1</text>
 <text x="-322.58" y="99.06" size="6.4516" layer="91">Vcc</text>
+<text x="167.64" y="-215.9" size="1.778" layer="91">Actually, swap
+these A&lt;-&gt;B</text>
+<text x="185.42" y="-254" size="1.778" layer="91">Actually, swap
+these A&lt;-&gt;B</text>
+<text x="287.02" y="-231.14" size="1.778" layer="91">RR</text>
+<text x="287.02" y="-254" size="1.778" layer="91">GG</text>
+<text x="287.02" y="-266.7" size="1.778" layer="91">BB</text>
+<text x="335.28" y="-261.62" size="1.778" layer="91">HSync</text>
+<text x="335.28" y="-269.24" size="1.778" layer="91">VSync</text>
+<text x="218.44" y="-289.56" size="1.778" layer="91">Always
+A -&gt; B</text>
+<text x="345.44" y="53.34" size="1.778" layer="91">VGA Blanker</text>
 </plain>
 <instances>
@@
 <instance part="INVERTOR" gate="A" x="-167.64" y="-147.32" rot="R270"/>
 <instance part="BUFFER3" gate="A" x="233.68" y="-256.54"/>
+<instance part="P+7" gate="1" x="213.36" y="-287.02" rot="R180"/>
+<instance part="GND8" gate="1" x="-121.92" y="-96.52" rot="R180"/>
+<instance part="GND9" gate="1" x="-83.82" y="-106.68" rot="R180"/>
+<instance part="GND15" gate="1" x="-45.72" y="-106.68" rot="R180"/>
+<instance part="GND16" gate="1" x="-7.62" y="-106.68" rot="R180"/>
+<instance part="GND17" gate="1" x="53.34" y="-170.18" rot="R180"/>
+<instance part="GND18" gate="1" x="38.1" y="-111.76" rot="R180"/>
+<instance part="GND19" gate="1" x="83.82" y="-109.22" rot="R180"/>
+<instance part="GND20" gate="1" x="121.92" y="-109.22" rot="R180"/>
+<instance part="GND21" gate="1" x="160.02" y="-109.22" rot="R180"/>
 </instances>
 <busses>
@@
 <pinref part="CONTROL" gate="A" pin="1B"/>
 <wire x1="30.48" y1="-175.26" x2="30.48" y2="-182.88" width="0.1524" layer="91"/>
+</segment>
+<segment>
+<pinref part="P+7" gate="1" pin="+5V"/>
+<wire x1="223.52" y1="-266.7" x2="213.36" y2="-266.7" width="0.1524" layer="91"/>
+<wire x1="213.36" y1="-266.7" x2="213.36" y2="-284.48" width="0.1524" layer="91"/>
 </segment>
 </net>
@@
 <wire x1="35.56" y1="-182.88" x2="35.56" y2="-157.48" width="0.1524" layer="91"/>
 </segment>
+<segment>
+<pinref part="MUX1" gate="A" pin="G"/>
+<pinref part="GND8" gate="1" pin="GND"/>
+<wire x1="-121.92" y1="-121.92" x2="-121.92" y2="-99.06" width="0.1524" layer="91"/>
+</segment>
+<segment>
+<pinref part="GND9" gate="1" pin="GND"/>
+<pinref part="MUX2" gate="A" pin="G"/>
+<wire x1="-83.82" y1="-109.22" x2="-83.82" y2="-121.92" width="0.1524" layer="91"/>
+</segment>
+<segment>
+<pinref part="GND15" gate="1" pin="GND"/>
+<pinref part="MUX3" gate="A" pin="G"/>
+<wire x1="-45.72" y1="-109.22" x2="-45.72" y2="-121.92" width="0.1524" layer="91"/>
+</segment>
+<segment>
+<pinref part="GND16" gate="1" pin="GND"/>
+<pinref part="MUX4" gate="A" pin="G"/>
+<wire x1="-7.62" y1="-109.22" x2="-7.62" y2="-121.92" width="0.1524" layer="91"/>
+</segment>
+<segment>
+<pinref part="GND18" gate="1" pin="GND"/>
+<wire x1="38.1" y1="-114.3" x2="38.1" y2="-121.92" width="0.1524" layer="91"/>
+</segment>
+<segment>
+<pinref part="GND19" gate="1" pin="GND"/>
+<pinref part="MUX6" gate="A" pin="G"/>
+<wire x1="83.82" y1="-111.76" x2="83.82" y2="-121.92" width="0.1524" layer="91"/>
+</segment>
+<segment>
+<pinref part="GND20" gate="1" pin="GND"/>
+<pinref part="MUX7" gate="A" pin="G"/>
+<wire x1="121.92" y1="-111.76" x2="121.92" y2="-121.92" width="0.1524" layer="91"/>
+</segment>
+<segment>
+<pinref part="GND21" gate="1" pin="GND"/>
+<pinref part="MUX8" gate="A" pin="G"/>
+<wire x1="160.02" y1="-111.76" x2="160.02" y2="-121.92" width="0.1524" layer="91"/>
+</segment>
+<segment>
+<pinref part="GND17" gate="1" pin="GND"/>
+<pinref part="CONTROL" gate="A" pin="G"/>
+<wire x1="53.34" y1="-172.72" x2="53.34" y2="-182.88" width="0.1524" layer="91"/>
+</segment>
 </net>
 <net name="N$1" class="0">
@@
 <pinref part="R3" gate="G$1" pin="1"/>
 <wire x1="279.4" y1="-236.22" x2="284.48" y2="-236.22" width="0.1524" layer="91"/>
-<wire x1="284.48" y1="-236.22" x2="284.48" y2="-238.76" width="0.1524" layer="91"/>
-<pinref part="X1" gate="-3" pin="F"/>
-<wire x1="284.48" y1="-238.76" x2="297.18" y2="-238.76" width="0.1524" layer="91"/>
 <pinref part="R4" gate="G$1" pin="1"/>
 <wire x1="279.4" y1="-241.3" x2="284.48" y2="-241.3" width="0.1524" layer="91"/>
 <wire x1="284.48" y1="-241.3" x2="284.48" y2="-238.76" width="0.1524" layer="91"/>
+<pinref part="X1" gate="-1" pin="F"/>
+<wire x1="284.48" y1="-238.76" x2="284.48" y2="-236.22" width="0.1524" layer="91"/>
+<wire x1="297.18" y1="-233.68" x2="287.02" y2="-233.68" width="0.1524" layer="91"/>
+<wire x1="287.02" y1="-233.68" x2="287.02" y2="-238.76" width="0.1524" layer="91"/>
+<wire x1="287.02" y1="-238.76" x2="284.48" y2="-238.76" width="0.1524" layer="91"/>
 <junction x="284.48" y="-238.76"/>
 </segment>
@@
 <pinref part="R5" gate="G$1" pin="1"/>
 <wire x1="279.4" y1="-248.92" x2="284.48" y2="-248.92" width="0.1524" layer="91"/>
-<wire x1="284.48" y1="-248.92" x2="284.48" y2="-251.46" width="0.1524" layer="91"/>
-<pinref part="X1" gate="-8" pin="F"/>
-<wire x1="284.48" y1="-251.46" x2="297.18" y2="-251.46" width="0.1524" layer="91"/>
 <pinref part="R6" gate="G$1" pin="1"/>
 <wire x1="279.4" y1="-254" x2="284.48" y2="-254" width="0.1524" layer="91"/>
 <wire x1="284.48" y1="-254" x2="284.48" y2="-251.46" width="0.1524" layer="91"/>
+<pinref part="X1" gate="-2" pin="F"/>
+<wire x1="284.48" y1="-251.46" x2="284.48" y2="-248.92" width="0.1524" layer="91"/>
+<wire x1="297.18" y1="-236.22" x2="289.56" y2="-236.22" width="0.1524" layer="91"/>
+<wire x1="289.56" y1="-236.22" x2="289.56" y2="-251.46" width="0.1524" layer="91"/>
+<wire x1="289.56" y1="-251.46" x2="284.48" y2="-251.46" width="0.1524" layer="91"/>
 <junction x="284.48" y="-251.46"/>
 </segment>
@@
 <pinref part="R7" gate="G$1" pin="1"/>
 <wire x1="279.4" y1="-261.62" x2="284.48" y2="-261.62" width="0.1524" layer="91"/>
-<wire x1="284.48" y1="-261.62" x2="284.48" y2="-264.16" width="0.1524" layer="91"/>
-<pinref part="X1" gate="-13" pin="F"/>
-<wire x1="284.48" y1="-264.16" x2="297.18" y2="-264.16" width="0.1524" layer="91"/>
 <pinref part="R8" gate="G$1" pin="1"/>
 <wire x1="279.4" y1="-266.7" x2="284.48" y2="-266.7" width="0.1524" layer="91"/>
 <wire x1="284.48" y1="-266.7" x2="284.48" y2="-264.16" width="0.1524" layer="91"/>
+<pinref part="X1" gate="-3" pin="F"/>
+<wire x1="284.48" y1="-264.16" x2="284.48" y2="-261.62" width="0.1524" layer="91"/>
+<wire x1="297.18" y1="-238.76" x2="292.1" y2="-238.76" width="0.1524" layer="91"/>
+<wire x1="292.1" y1="-238.76" x2="292.1" y2="-264.16" width="0.1524" layer="91"/>
+<wire x1="292.1" y1="-264.16" x2="284.48" y2="-264.16" width="0.1524" layer="91"/>
 <junction x="284.48" y="-264.16"/>
+</segment>
+</net>
+<net name="N$122" class="0">
+<segment>
+<pinref part="X1" gate="-13" pin="F"/>
+<wire x1="297.18" y1="-264.16" x2="342.9" y2="-264.16" width="0.1524" layer="91"/>
+<wire x1="342.9" y1="-264.16" x2="342.9" y2="50.8" width="0.1524" layer="91"/>
+<pinref part="GPU" gate="G$1" pin="PCINT1/ADC1_PA1"/>
+<wire x1="342.9" y1="50.8" x2="304.8" y2="50.8" width="0.1524" layer="91"/>
+</segment>
+</net>
+<net name="N$124" class="0">
+<segment>
+<pinref part="X1" gate="-14" pin="F"/>
+<wire x1="297.18" y1="-266.7" x2="345.44" y2="-266.7" width="0.1524" layer="91"/>
+<wire x1="345.44" y1="-266.7" x2="345.44" y2="48.26" width="0.1524" layer="91"/>
+<pinref part="GPU" gate="G$1" pin="PCINT2/ADC2_PA2"/>
+<wire x1="345.44" y1="48.26" x2="304.8" y2="48.26" width="0.1524" layer="91"/>
+</segment>
+</net>
+<net name="N$125" class="0">
+<segment>
+<pinref part="BUFFER3" gate="A" pin="G"/>
+<wire x1="220.98" y1="-269.24" x2="220.98" y2="-276.86" width="0.1524" layer="91"/>
+<wire x1="220.98" y1="-276.86" x2="353.06" y2="-276.86" width="0.1524" layer="91"/>
+<wire x1="353.06" y1="-276.86" x2="353.06" y2="53.34" width="0.1524" layer="91"/>
+<pinref part="GPU" gate="G$1" pin="PCINT0/ADC0_PA0"/>
+<wire x1="353.06" y1="53.34" x2="304.8" y2="53.34" width="0.1524" layer="91"/>
 </segment>
 </net>
@@
 </schematic>
 </drawing>
+<compatibility>
+<note version="6.3" minversion="6.2.2" severity="warning">
+Since Version 6.2.2 text objects can contain more than one line,
+which will not be processed correctly with this version.
+</note>
+</compatibility>
 </eagle>

Commit message: VRAM schematic update, nailing pins down
Parts:
- added C6, C7, C8, C9: 22pF, capacitor-wima:C2,5-3
Connections:
- new net N$120: C8.2, IC2.XTAL2, Q1.1
- new net N$126: C9.2, IC2.XTAL1, Q1.2
- new net N$128: BUFFER1A.DIR, BUFFER2A.DIR, IC2.PG2(ALE)
- net GND: now also C8.1, C9.1; no longer IC2.XTAL1, IC2.XTAL2, Q1.1, Q1.2
- net N$2: now also IC2.PG1(RD); no longer IC2.PG2(ALE)
- net N$3: now also IC2.PG0(WR); no longer IC2.PG1(RD)
Other:
- note added: "VRAMA"
- note added: "VRAMB"
- note removed: "RAMA"
- note removed: "RAMB"
- moved on the sheet: RS232-CPU, SERIALCPU
Changed lines of the file:
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@@
 <part name="GND20" library="supply1" deviceset="GND" device=""/>
 <part name="GND21" library="supply1" deviceset="GND" device=""/>
+<part name="C6" library="capacitor-wima" deviceset="C" device="2,5-3" value="22pF"/>
+<part name="C7" library="capacitor-wima" deviceset="C" device="2,5-3" value="22pF"/>
+<part name="C8" library="capacitor-wima" deviceset="C" device="2,5-3" value="22pF"/>
+<part name="C9" library="capacitor-wima" deviceset="C" device="2,5-3" value="22pF"/>
 </parts>
 <sheets>
 <sheet>
 <plain>
-<text x="-109.22" y="-180.34" size="6.4516" layer="91">RAMA</text>
-<text x="144.78" y="-180.34" size="6.4516" layer="91">RAMB</text>
-<text x="-162.56" y="-129.54" size="6.4516" layer="91">DATAA</text>
-<text x="-200.66" y="-129.54" size="6.4516" layer="91">DATAB</text>
+<text x="-114.3" y="-185.42" size="6.4516" layer="91">VRAMA</text>
+<text x="144.78" y="-185.42" size="6.4516" layer="91">VRAMB</text>
+<text x="-162.56" y="-134.62" size="6.4516" layer="91">DATAA</text>
+<text x="-200.66" y="-134.62" size="6.4516" layer="91">DATAB</text>
 <text x="22.86" y="-220.98" size="3.81" layer="91">RAM CTRL SW</text>
 <text x="-246.38" y="86.36" size="6.4516" layer="91">CPU</text>
@@
 <instance part="MUX10" gate="A" x="175.26" y="-236.22"/>
 <instance part="IC2" gate="G$1" x="-236.22" y="25.4"/>
-<instance part="RS232-CPU" gate="G$1" x="-271.78" y="-68.58"/>
+<instance part="RS232-CPU" gate="G$1" x="-246.38" y="-68.58"/>
 <instance part="RS232-GPU" gate="G$1" x="215.9" y="73.66"/>
-<instance part="GND10" gate="1" x="-281.94" y="71.12" rot="R270"/>
+<instance part="GND10" gate="1" x="-294.64" y="71.12" rot="R270"/>
 <instance part="JP2" gate="G$1" x="-274.32" y="7.62" rot="R180"/>
 <instance part="GND11" gate="1" x="-297.18" y="10.16" rot="R270"/>
 <instance part="P+9" gate="1" x="-299.72" y="5.08" rot="R90"/>
-<instance part="SERIALCPU" gate="G$1" x="-304.8" y="-78.74"/>
+<instance part="SERIALCPU" gate="G$1" x="-279.4" y="-78.74"/>
 <instance part="SERIALGPU" gate="G$1" x="182.88" y="63.5"/>
 <instance part="JOY1" gate="G$1" x="-81.28" y="104.14" rot="R270"/>
@@
 <instance part="GND20" gate="1" x="121.92" y="-109.22" rot="R180"/>
 <instance part="GND21" gate="1" x="160.02" y="-109.22" rot="R180"/>
+<instance part="C6" gate="G$1" x="228.6" y="25.4" rot="MR270"/>
+<instance part="C7" gate="G$1" x="220.98" y="22.86" rot="MR270"/>
+<instance part="C8" gate="G$1" x="-284.48" y="73.66" rot="MR270"/>
+<instance part="C9" gate="G$1" x="-284.48" y="68.58" rot="MR270"/>
 </instances>
 <busses>
@@
 <wire x1="320.04" y1="25.4" x2="332.74" y2="25.4" width="0.1524" layer="91"/>
 <junction x="320.04" y="25.4"/>
-</segment>
-<segment>
-<pinref part="GND10" gate="1" pin="GND"/>
-<wire x1="-279.4" y1="71.12" x2="-279.4" y2="73.66" width="0.1524" layer="91"/>
-<pinref part="IC2" gate="G$1" pin="XTAL2"/>
-<pinref part="Q1" gate="G$1" pin="1"/>
-<wire x1="-264.16" y1="73.66" x2="-271.78" y2="73.66" width="0.1524" layer="91"/>
-<wire x1="-279.4" y1="73.66" x2="-271.78" y2="73.66" width="0.1524" layer="91"/>
-<pinref part="IC2" gate="G$1" pin="XTAL1"/>
-<pinref part="Q1" gate="G$1" pin="2"/>
-<wire x1="-264.16" y1="68.58" x2="-271.78" y2="68.58" width="0.1524" layer="91"/>
-<wire x1="-279.4" y1="71.12" x2="-279.4" y2="68.58" width="0.1524" layer="91"/>
-<wire x1="-279.4" y1="68.58" x2="-271.78" y2="68.58" width="0.1524" layer="91"/>
 </segment>
 <segment>
@@
 <wire x1="53.34" y1="-172.72" x2="53.34" y2="-182.88" width="0.1524" layer="91"/>
 </segment>
+<segment>
+<pinref part="C8" gate="G$1" pin="1"/>
+<wire x1="-287.02" y1="73.66" x2="-292.1" y2="73.66" width="0.1524" layer="91"/>
+<pinref part="GND10" gate="1" pin="GND"/>
+<wire x1="-292.1" y1="73.66" x2="-292.1" y2="71.12" width="0.1524" layer="91"/>
+<wire x1="-292.1" y1="71.12" x2="-292.1" y2="68.58" width="0.1524" layer="91"/>
+<pinref part="C9" gate="G$1" pin="1"/>
+<wire x1="-292.1" y1="68.58" x2="-287.02" y2="68.58" width="0.1524" layer="91"/>
+<junction x="-292.1" y="71.12"/>
+</segment>
 </net>
 <net name="N$1" class="0">
@@
 <wire x1="45.72" y1="-12.7" x2="33.02" y2="-12.7" width="0.1524" layer="91"/>
 <junction x="33.02" y="-12.7"/>
-<wire x1="-307.34" y1="-45.72" x2="-307.34" y2="30.48" width="0.1524" layer="91"/>
-<pinref part="IC2" gate="G$1" pin="PG2(ALE)"/>
-<wire x1="-307.34" y1="30.48" x2="-264.16" y2="30.48" width="0.1524" layer="91"/>
+<wire x1="-307.34" y1="-45.72" x2="-307.34" y2="27.94" width="0.1524" layer="91"/>
 <wire x1="-307.34" y1="-45.72" x2="-127" y2="-45.72" width="0.1524" layer="91"/>
 <wire x1="-127" y1="-45.72" x2="-127" y2="-12.7" width="0.1524" layer="91"/>
+<pinref part="IC2" gate="G$1" pin="PG1(RD)"/>
+<wire x1="-264.16" y1="27.94" x2="-307.34" y2="27.94" width="0.1524" layer="91"/>
 </segment>
 </net>
@@
 <net name="N$3" class="0">
 <segment>
-<pinref part="IC2" gate="G$1" pin="PG1(RD)"/>
-<wire x1="-309.88" y1="-48.26" x2="-309.88" y2="27.94" width="0.1524" layer="91"/>
-<wire x1="-309.88" y1="27.94" x2="-264.16" y2="27.94" width="0.1524" layer="91"/>
+<wire x1="-309.88" y1="-48.26" x2="-309.88" y2="25.4" width="0.1524" layer="91"/>
 <pinref part="CONTROL" gate="A" pin="1A"/>
 <wire x1="27.94" y1="-182.88" x2="27.94" y2="-15.24" width="0.1524" layer="91"/>
@@
 <wire x1="-309.88" y1="-48.26" x2="-124.46" y2="-48.26" width="0.1524" layer="91"/>
 <wire x1="-124.46" y1="-48.26" x2="-124.46" y2="-15.24" width="0.1524" layer="91"/>
+<pinref part="IC2" gate="G$1" pin="PG0(WR)"/>
+<wire x1="-264.16" y1="25.4" x2="-309.88" y2="25.4" width="0.1524" layer="91"/>
 </segment>
 </net>
@@
 </segment>
 </net>
+<net name="N$120" class="0">
+<segment>
+<pinref part="Q1" gate="G$1" pin="1"/>
+<wire x1="-279.4" y1="73.66" x2="-271.78" y2="73.66" width="0.1524" layer="91"/>
+<pinref part="IC2" gate="G$1" pin="XTAL2"/>
+<wire x1="-264.16" y1="73.66" x2="-271.78" y2="73.66" width="0.1524" layer="91"/>
+<pinref part="C8" gate="G$1" pin="2"/>
+</segment>
+</net>
+<net name="N$126" class="0">
+<segment>
+<pinref part="IC2" gate="G$1" pin="XTAL1"/>
+<pinref part="Q1" gate="G$1" pin="2"/>
+<wire x1="-264.16" y1="68.58" x2="-271.78" y2="68.58" width="0.1524" layer="91"/>
+<wire x1="-279.4" y1="68.58" x2="-271.78" y2="68.58" width="0.1524" layer="91"/>
+<pinref part="C9" gate="G$1" pin="2"/>
+</segment>
+</net>
+<net name="N$128" class="0">
+<segment>
+<pinref part="BUFFER1" gate="A" pin="DIR"/>
+<wire x1="-134.62" y1="-119.38" x2="-134.62" y2="-121.92" width="0.1524" layer="91"/>
+<pinref part="BUFFER2" gate="A" pin="DIR"/>
+<wire x1="-172.72" y1="-119.38" x2="-172.72" y2="-121.92" width="0.1524" layer="91"/>
+<wire x1="-134.62" y1="-121.92" x2="-172.72" y2="-121.92" width="0.1524" layer="91"/>
+<wire x1="-172.72" y1="-121.92" x2="-312.42" y2="-121.92" width="0.1524" layer="91"/>
+<wire x1="-312.42" y1="-121.92" x2="-312.42" y2="30.48" width="0.1524" layer="91"/>
+<pinref part="IC2" gate="G$1" pin="PG2(ALE)"/>
+<wire x1="-312.42" y1="30.48" x2="-264.16" y2="30.48" width="0.1524" layer="91"/>
+</segment>
+</net>

Commit message: Added resistor values to zz r3 schem
Other:
- note added: "1K"
- note added: "2K"
- note added: "HIGH"
- note added: "LOW"
Changed lines of the file:
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@@
 A -&gt; B</text>
 <text x="345.44" y="53.34" size="1.778" layer="91">VGA Blanker</text>
+<text x="-7.62" y="-139.7" size="1.778" layer="91">LOW</text>
+<text x="-45.72" y="-139.7" size="1.778" layer="91">LOW</text>
+<text x="-83.82" y="-139.7" size="1.778" layer="91">HIGH</text>
+<text x="-121.92" y="-139.7" size="1.778" layer="91">HIGH</text>
+<text x="160.02" y="-139.7" size="1.778" layer="91">LOW</text>
+<text x="121.92" y="-139.7" size="1.778" layer="91">LOW</text>
+<text x="48.26" y="-139.7" size="1.778" layer="91">HIGH</text>
+<text x="83.82" y="-139.7" size="1.778" layer="91">HIGH</text>
+<text x="269.24" y="-233.68" size="1.778" layer="91">1K</text>
+<text x="269.24" y="-246.38" size="1.778" layer="91">1K</text>
+<text x="269.24" y="-259.08" size="1.778" layer="91">1K</text>
+<text x="279.4" y="-243.84" size="1.778" layer="91">2K</text>
+<text x="279.4" y="-256.54" size="1.778" layer="91">2K</text>
+<text x="279.4" y="-269.24" size="1.778" layer="91">2K</text>
 </plain>
 <instances>
