File: zikzak5-zikz80/schem/zikzak-z80-2.sch (EAGLE design)
At the start: 65 parts, among them IC1 Z80, IC10 74LS32N, IC11 74LS32N, IC12 74LS32N, IC13 74LS32N, IC14 74LS04N, IC15 74LS32N, IC16 ATMEGA644-20PU, IC2 ATMEGA644-20PU, IC3 MC6850, IC4 74LS32N, IC5 74LS04N, IC6 74LS32N, U2 FT232RLSSOP, X2 USB-SMD-NS

Commit message: Updated schem
Parts:
- added JP1: ISP, pinhead:PINHD-1X6
Connections:
- new net IO_MISO: IC16.PCINT14/MISO_PB6, JP1.1
- new net IO_MOSI: IC16.PCINT13/MOSI_PB5, JP1.4
- new net IO_RESET: IC16.!RESET, JP1.5
- new net IO_SCK: IC16.PCINT15/SCK_PB7, JP1.3
- net 5V: now also JP1.2
- net AT_MISO: no longer IC16.PCINT14/MISO_PB6
- net AT_MOSI: no longer IC16.PCINT13/MOSI_PB5
- net AT_RESET: no longer IC16.!RESET
- net AT_SCK: no longer IC16.PCINT15/SCK_PB7
- net GND: now also JP1.6
Other:
- note added: "ISP Progr. IO"
- note added: "ISP Progr. VGA"
- note added: "TODO: - color VGA DAC - color / mono switch via buffer IC? - audio DAC .. mnaybe via Shift Register? - add pull up on avr /RESET * 2"
- note removed: "ISP Progr."
- note removed: "TODO: - color VGA DAC - color / mono switch via buffer IC? - audio DAC"
- moved on the sheet: JP2
Changed lines of the file:
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@@
 <part name="GND14" library="SparkFun" deviceset="GND" device=""/>
 <part name="C12" library="rcl" deviceset="C-EU" device="025-050X050"/>
+<part name="JP1" library="pinhead" deviceset="PINHD-1X6" device="" value="ISP"/>
 </parts>
 <sheets>
@@
 <text x="273.05" y="80.01" size="1.27" layer="91">/</text>
 <text x="273.05" y="77.47" size="1.27" layer="91">/</text>
-<rectangle x1="5.08" y1="116.84" x2="36.83" y2="143.51" layer="203"/>
+<rectangle x1="5.08" y1="157.48" x2="36.83" y2="184.15" layer="203"/>
 <text x="320.04" y="45.72" size="5.08" layer="91">VGA</text>
 <text x="15.24" y="29.21" size="5.08" layer="91">PS/2 Keyb</text>
-<text x="7.62" y="146.05" size="5.08" layer="91">ISP Progr.</text>
+<text x="7.62" y="186.69" size="5.08" layer="91">ISP Progr. VGA</text>
 <text x="76.2" y="191.77" size="5.08" layer="91">Serial &lt;-&gt; USB</text>
 <text x="354.33" y="72.39" size="1.016" layer="91">decoupling
@@
 <text x="417.83" y="100.33" size="5.08" layer="91">VGA Gen</text>
 <text x="405.13" y="228.6" size="5.08" layer="91">IO/CLK/SID</text>
-<text x="419.1" y="121.92" size="6.4516" layer="91">TODO:
+<text x="445.77" y="129.54" size="3.81" layer="94">TODO:
 - color VGA DAC
 -   color / mono switch via buffer IC?
-- audio DAC</text>
+- audio DAC .. mnaybe via Shift Register?
+- add pull up on avr /RESET * 2</text>
+<rectangle x1="3.81" y1="109.22" x2="35.56" y2="135.89" layer="203"/>
+<text x="6.35" y="138.43" size="5.08" layer="91">ISP Progr. IO</text>
 </plain>
 <instances>
@@
 <instance part="GND8" gate="1" x="38.354" y="220.472"/>
 <instance part="U$3" gate="G$1" x="56.134" y="250.952"/>
-<instance part="JP2" gate="A" x="9.398" y="131.572" rot="R180"/>
+<instance part="JP2" gate="A" x="9.398" y="172.212" rot="R180"/>
 <instance part="GND6" gate="1" x="112.014" y="256.032" rot="R180"/>
 <instance part="IC2" gate="G$1" x="428.498" y="72.39"/>
@@
 <instance part="GND14" gate="1" x="379.73" y="259.08" rot="R180"/>
 <instance part="C12" gate="G$1" x="483.108" y="198.882"/>
+<instance part="JP1" gate="A" x="8.128" y="123.952" rot="R180"/>
 </instances>
 <busses>
@@
 <segment>
 <pinref part="JP2" gate="A" pin="6"/>
-<wire x1="11.938" y1="136.652" x2="22.098" y2="136.652" width="0.1524" layer="91"/>
-<label x="22.098" y="136.652" size="1.27" layer="95" xref="yes"/>
+<wire x1="11.938" y1="177.292" x2="22.098" y2="177.292" width="0.1524" layer="91"/>
+<label x="22.098" y="177.292" size="1.27" layer="95" xref="yes"/>
 </segment>
 <segment>
@@
 <junction x="379.73" y="256.54"/>
 </segment>
+<segment>
+<pinref part="JP1" gate="A" pin="6"/>
+<wire x1="10.668" y1="129.032" x2="20.828" y2="129.032" width="0.1524" layer="91"/>
+<label x="20.828" y="129.032" size="1.27" layer="95" xref="yes"/>
+</segment>
 </net>
 <net name="USB_D-" class="0">
@@
 <segment>
 <pinref part="JP2" gate="A" pin="2"/>
-<wire x1="11.938" y1="126.492" x2="22.098" y2="126.492" width="0.1524" layer="91"/>
-<label x="22.098" y="126.492" size="1.27" layer="95" xref="yes"/>
+<wire x1="11.938" y1="167.132" x2="22.098" y2="167.132" width="0.1524" layer="91"/>
+<label x="22.098" y="167.132" size="1.27" layer="95" xref="yes"/>
 </segment>
 <segment>
@@
 <junction x="455.168" y="198.12"/>
 </segment>
+<segment>
+<pinref part="JP1" gate="A" pin="2"/>
+<wire x1="10.668" y1="118.872" x2="20.828" y2="118.872" width="0.1524" layer="91"/>
+<label x="20.828" y="118.872" size="1.27" layer="95" xref="yes"/>
+</segment>
 </net>
 <net name="AT_MOSI" class="0">
 <segment>
 <pinref part="JP2" gate="A" pin="4"/>
-<wire x1="11.938" y1="131.572" x2="22.098" y2="131.572" width="0.1524" layer="91"/>
-<label x="22.098" y="131.572" size="1.27" layer="95" xref="yes"/>
+<wire x1="11.938" y1="172.212" x2="22.098" y2="172.212" width="0.1524" layer="91"/>
+<label x="22.098" y="172.212" size="1.27" layer="95" xref="yes"/>
 </segment>
 <segment>
@@
 <junction x="253.492" y="26.67"/>
 </segment>
-<segment>
-<wire x1="394.97" y1="210.82" x2="394.208" y2="210.82" width="0.1524" layer="91"/>
-<label x="388.62" y="210.82" size="1.27" layer="95" rot="R180" xref="yes"/>
-<pinref part="IC16" gate="G$1" pin="PCINT13/MOSI_PB5"/>
-<wire x1="394.208" y1="210.82" x2="388.62" y2="210.82" width="0.1524" layer="91"/>
-<junction x="394.208" y="210.82"/>
-</segment>
 </net>
 <net name="AT_SCK" class="0">
 <segment>
 <pinref part="JP2" gate="A" pin="3"/>
-<wire x1="11.938" y1="129.032" x2="22.098" y2="129.032" width="0.1524" layer="91"/>
-<label x="22.098" y="129.032" size="1.27" layer="95" xref="yes"/>
+<wire x1="11.938" y1="169.672" x2="22.098" y2="169.672" width="0.1524" layer="91"/>
+<label x="22.098" y="169.672" size="1.27" layer="95" xref="yes"/>
 </segment>
 <segment>
@@
 <junction x="398.018" y="77.47"/>
 </segment>
-<segment>
-<wire x1="394.97" y1="205.74" x2="394.208" y2="205.74" width="0.1524" layer="91"/>
-<label x="388.62" y="205.74" size="1.27" layer="95" rot="R180" xref="yes"/>
-<pinref part="IC16" gate="G$1" pin="PCINT15/SCK_PB7"/>
-<wire x1="394.208" y1="205.74" x2="388.62" y2="205.74" width="0.1524" layer="91"/>
-<junction x="394.208" y="205.74"/>
-</segment>
 </net>
 <net name="AT_MISO" class="0">
 <segment>
 <pinref part="JP2" gate="A" pin="1"/>
-<wire x1="11.938" y1="123.952" x2="22.098" y2="123.952" width="0.1524" layer="91"/>
-<label x="22.098" y="123.952" size="1.27" layer="95" xref="yes"/>
+<wire x1="11.938" y1="164.592" x2="22.098" y2="164.592" width="0.1524" layer="91"/>
+<label x="22.098" y="164.592" size="1.27" layer="95" xref="yes"/>
 </segment>
 <segment>
@@
 <wire x1="239.522" y1="21.59" x2="238.76" y2="21.59" width="0.1524" layer="91"/>
 <junction x="239.522" y="21.59"/>
-</segment>
-<segment>
-<wire x1="394.97" y1="208.28" x2="394.208" y2="208.28" width="0.1524" layer="91"/>
-<label x="388.62" y="208.28" size="1.27" layer="95" rot="R180" xref="yes"/>
-<pinref part="IC16" gate="G$1" pin="PCINT14/MISO_PB6"/>
-<wire x1="394.208" y1="208.28" x2="388.62" y2="208.28" width="0.1524" layer="91"/>
-<junction x="394.208" y="208.28"/>
 </segment>
 </net>
@@
 <segment>
 <pinref part="JP2" gate="A" pin="5"/>
-<wire x1="11.938" y1="134.112" x2="22.098" y2="134.112" width="0.1524" layer="91"/>
-<label x="22.098" y="134.112" size="1.27" layer="95" xref="yes"/>
-</segment>
-<segment>
-<wire x1="394.97" y1="203.2" x2="394.208" y2="203.2" width="0.1524" layer="91"/>
-<label x="388.62" y="203.2" size="1.27" layer="95" rot="R180" xref="yes"/>
-<pinref part="IC16" gate="G$1" pin="!RESET"/>
-<wire x1="394.208" y1="203.2" x2="388.62" y2="203.2" width="0.1524" layer="91"/>
-<junction x="394.208" y="203.2"/>
+<wire x1="11.938" y1="174.752" x2="22.098" y2="174.752" width="0.1524" layer="91"/>
+<label x="22.098" y="174.752" size="1.27" layer="95" xref="yes"/>
 </segment>
 </net>
@@
 </segment>
 </net>
+<net name="IO_RESET" class="0">
+<segment>
+<pinref part="JP1" gate="A" pin="5"/>
+<wire x1="10.668" y1="126.492" x2="20.828" y2="126.492" width="0.1524" layer="91"/>
+<label x="20.828" y="126.492" size="1.27" layer="95" xref="yes"/>
+</segment>
+<segment>
+<wire x1="394.97" y1="203.2" x2="394.208" y2="203.2" width="0.1524" layer="91"/>
+<label x="388.62" y="203.2" size="1.27" layer="95" rot="R180" xref="yes"/>
+<pinref part="IC16" gate="G$1" pin="!RESET"/>
+<wire x1="394.208" y1="203.2" x2="388.62" y2="203.2" width="0.1524" layer="91"/>
+<junction x="394.208" y="203.2"/>
+</segment>
+</net>
+<net name="IO_MOSI" class="0">
+<segment>
+<pinref part="JP1" gate="A" pin="4"/>
+<wire x1="10.668" y1="123.952" x2="20.828" y2="123.952" width="0.1524" layer="91"/>
+<label x="20.828" y="123.952" size="1.27" layer="95" xref="yes"/>
+</segment>
+<segment>
+<wire x1="394.97" y1="210.82" x2="394.208" y2="210.82" width="0.1524" layer="91"/>
+<label x="388.62" y="210.82" size="1.27" layer="95" rot="R180" xref="yes"/>
+<pinref part="IC16" gate="G$1" pin="PCINT13/MOSI_PB5"/>
+<wire x1="394.208" y1="210.82" x2="388.62" y2="210.82" width="0.1524" layer="91"/>
+<junction x="394.208" y="210.82"/>
+</segment>
+</net>
+<net name="IO_SCK" class="0">
+<segment>
+<pinref part="JP1" gate="A" pin="3"/>
+<wire x1="10.668" y1="121.412" x2="20.828" y2="121.412" width="0.1524" layer="91"/>
+<label x="20.828" y="121.412" size="1.27" layer="95" xref="yes"/>
+</segment>
+<segment>
+<wire x1="394.97" y1="205.74" x2="394.208" y2="205.74" width="0.1524" layer="91"/>
+<label x="388.62" y="205.74" size="1.27" layer="95" rot="R180" xref="yes"/>
+<pinref part="IC16" gate="G$1" pin="PCINT15/SCK_PB7"/>
+<wire x1="394.208" y1="205.74" x2="388.62" y2="205.74" width="0.1524" layer="91"/>
+<junction x="394.208" y="205.74"/>
+</segment>
+</net>
+<net name="IO_MISO" class="0">
+<segment>
+<pinref part="JP1" gate="A" pin="1"/>
+<wire x1="10.668" y1="116.332" x2="20.828" y2="116.332" width="0.1524" layer="91"/>
+<label x="20.828" y="116.332" size="1.27" layer="95" xref="yes"/>
+</segment>
+<segment>
+<wire x1="394.97" y1="208.28" x2="394.208" y2="208.28" width="0.1524" layer="91"/>
+<label x="388.62" y="208.28" size="1.27" layer="95" rot="R180" xref="yes"/>
+<pinref part="IC16" gate="G$1" pin="PCINT14/MISO_PB6"/>
+<wire x1="394.208" y1="208.28" x2="388.62" y2="208.28" width="0.1524" layer="91"/>
+<junction x="394.208" y="208.28"/>
+</segment>
+</net>
