File: zikcart/protocard_2x18/zikcart/zikcart-atc256-001.sch (EAGLE design)
At the start: 20 parts

Commit message: zikcart tweaked and brd layout done, and gerbers generated!
Connections:
- net _GND renamed GND
- net _VCC renamed VCC
