File: zikcart/protocard_2x18/zikcart/zikcart-atc256-001.brd (EAGLE design)
At the start: 73.6 x 55.5 mm, 20 parts

Commit message: zikcart tweaked and brd layout done, and gerbers generated!
Parts:
- moved C1 10.9 mm to (64.9, 16.3)
Connections:
- net _GND renamed GND
- net _VCC renamed VCC
Routing:
- net VCC: track 0.00 -> 98.7 mm
- net !WE!: track 0.00 -> 67.9 mm, vias 0 -> 2
- net A14: track 0.00 -> 54.4 mm, vias 0 -> 1
- net A12: track 0.00 -> 54.3 mm, vias 0 -> 1
- net A10: track 0.00 -> 54.2 mm, vias 0 -> 1
- net !OE!: track 0.00 -> 53.1 mm, vias 0 -> 1
- net !CE!: track 0.00 -> 52.1 mm, vias 0 -> 1
- net A11: track 0.00 -> 46.1 mm
- net IO2: track 0.00 -> 45.5 mm
- net A7: track 0.00 -> 45.0 mm
- net A6: track 0.00 -> 44.7 mm
- net A9: track 0.00 -> 44.3 mm, vias 0 -> 1
- net IO1: track 0.00 -> 44.1 mm
- net A5: track 0.00 -> 43.2 mm
- net A4: track 0.00 -> 42.6 mm
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- added copper zone on layer 1, net GND
- added copper zone on layer 16, net GND
Other:
- board text added: "Zikzak http://www.zikzak.ca Jeff Mitchell 2014"
- board text added: "rev 1"

Commit message: First board submission to elecrow! (on special, 50% off small boards)
Parts:
- moved AT28C256 7.62 mm to (38.1, 11.4)
- moved C1 7.62 mm to (64.9, 8.69)
- moved 1,19 7.62 mm to (1.19, 41.5)
- moved 10,28 7.62 mm to (36.9, 41.5)
- moved 11,29 7.62 mm to (40.8, 41.5)
- moved 12,30 7.62 mm to (44.8, 41.5)
- moved 13,31 7.62 mm to (48.7, 41.5)
- moved 14,32 7.62 mm to (52.7, 41.5)
- moved 15,33 7.62 mm to (56.7, 41.5)
- moved 16,34 7.62 mm to (60.6, 41.5)
- moved 17,35 7.62 mm to (64.6, 41.5)
- moved 18,36 7.62 mm to (68.5, 41.5)
- moved 2,20 7.62 mm to (5.15, 41.5)
- moved 3,21 7.62 mm to (9.11, 41.5)
- moved 4,22 7.62 mm to (13.1, 41.5)
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Other:
- board size 73.6 x 55.5 mm -> 73.6 x 47.9 mm
- board text added: "/CE GND"
- board text added: "/WE /OE"
- board text added: "A0 A21"
- board text added: "A1 A20"
- board text added: "A10 A11"
- board text added: "A2 A19"
- board text added: "A3 A18"
- board text added: "A4 A17"
- board text added: "A5 A16"
- board text added: "A6 A15"
- board text added: "A7 A14"
- board text added: "A8 A13"
- board text added: "A9 A12"
- board text added: "D0 D7"
- board text added: "D1 D6"
- board text added: "D2 D5"
- board text added: "D3 D4"
- board text added: "VCC33 VCC5"
- board text added: "Zikzak www.zikzak.ca Jeff Mitchell rev 1 02-2014"
- board text removed: "Zikzak http://www.zikzak.ca Jeff Mitchell 2014"
- board text removed: "rev 1"
