File: zik80/schem/zik-pcb-power.brd (EAGLE design)
At the start: 96.5 x 47.9 mm, 15 parts, among them IC1 TPS7133QP, IC2 7805TV, IC3 TPS7133QP

Commit message: rev1 of both power and gpu boards finalized, and elecrow gerber files generated!
Parts:
- moved R1 12.7 mm to (19.1, 35.6)
- moved IC1 2.84 mm to (64.8, 15.2), turned to 270 degrees
- moved IC3 2.84 mm to (64.8, 35.6), turned to 270 degrees
- moved U$2 2.84 mm to (27.9, 15.2)
- moved PWRIN 2.54 mm to (6.35, 6.35), turned to 90 degrees
- moved VCCIN 2.54 mm to (6.35, 34.3), turned to 90 degrees
- moved U$1 2.54 mm to (11.4, 20.3)
- moved LED1 1.80 mm to (25.4, 41.9), turned to 0 degrees
- moved C3 1.80 mm to (47.0, 11.4)
- moved PWROUT 1.80 mm to (90.2, 10.2)
- moved C2 1.27 mm to (77.5, 15.2)
- moved C1 1.27 mm to (77.5, 35.6)
- moved C4 1.27 mm to (47.0, 38.1)
- moved PWROUT2 1.27 mm to (90.2, 38.1)
Routing:
- net +5V: track 0.00 -> 191.1 mm
- net VCC: track 0.00 -> 112.8 mm
- net N$1: track 0.00 -> 39.2 mm
- net +3V3: track 0.00 -> 30.0 mm
- net V+: track 0.00 -> 27.4 mm
- net N$3: track 0.00 -> 6.35 mm
- added copper zone on layer 16, net GND
Other:
- board text added: "GND 3.3 5 VCC"
- board text added: "GND NC VCC5"
- board text added: "GND NC VCC9"
- board text added: "NC VCC9 GND"
- board text added: "PWRIN/JACK or (not both) VCCIN"
- board text added: "Zikzak www.zikzak.ca Jeff Mitchell Power rev 1 05-2014"

Commit message: Made a couple notes on power and gpu schems, of things needing correction; fiddled with vga out on real pcb.. works!
Parts:
- R1: value 1K -> 330 ohm
Changed lines of the file:
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@@
 <element name="VCCIN" library="pinhead" package="1X03" value="" x="6.35" y="34.29" rot="R90"/>
 <element name="LED1" library="SparkFun-LED" package="LED5MM" value="" x="25.4" y="41.91"/>
-<element name="R1" library="rcl" package="0207/10" value="1K" x="19.05" y="35.56"/>
+<element name="R1" library="rcl" package="0207/10" value="330 ohm" x="19.05" y="35.56"/>
 </elements>
 <signals>
