File: zik80/schem/zik-pcb-gpu-f405.brd (EAGLE design)
At the start: 99 x 98.7 mm, 48 parts

Commit message: GPU rev2 designed, ready to send up to elecrow .. *fear*
Connections:
- net NRST: now also ISPJTAG.15
- net PB4: no longer ISPJTAG.15
Routing:
- net PB4: track 39.1 -> 37.3 mm
Changed lines of the file:
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@@
 <?xml version="1.0" encoding="utf-8"?>
 <!DOCTYPE eagle SYSTEM "eagle.dtd">
-<eagle version="6.4">
+<eagle version="6.5.0">
 <drawing>
 <settings>
@@
 </signal>
 <signal name="PB4">
-<contactref element="ISPJTAG" pad="15"/>
 <contactref element="U$1" pad="56"/>
 <contactref element="JP4" pad="8"/>
@@
 <wire x1="32.385" y1="85.725" x2="31.75" y2="86.36" width="0.3048" layer="16"/>
 <wire x1="31.75" y1="86.36" x2="31.75" y2="90.17" width="0.3048" layer="16"/>
-<wire x1="31.75" y1="90.17" x2="30.48" y2="91.44" width="0.3048" layer="16"/>
 </signal>
 <signal name="PH1">
@@
 <wire x1="17.145" y1="54.61" x2="15.875" y2="55.88" width="0.3048" layer="1"/>
 <wire x1="15.875" y1="55.88" x2="13.97" y2="55.88" width="0.3048" layer="1"/>
+<contactref element="ISPJTAG" pad="15"/>
+<wire x1="15.875" y1="55.88" x2="30.48" y2="91.44" width="0" layer="19" extent="1-1"/>
 </signal>
 <signal name="PC0">
