File: zik80/schem/zik-pcb-gpu-f405.sch (EAGLE design)
At the start: 48 parts

Commit message: GPU rev2 designed, ready to send up to elecrow .. *fear*
Connections:
- net NRST: now also ISPJTAG.15
- net PB4: no longer ISPJTAG.15
Changed lines of the file:
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@@
 <?xml version="1.0" encoding="utf-8"?>
 <!DOCTYPE eagle SYSTEM "eagle.dtd">
-<eagle version="6.4">
+<eagle version="6.5.0">
 <drawing>
 <settings>
@@
 <net name="PB4" class="0">
 <segment>
-<pinref part="ISPJTAG" gate="A" pin="15"/>
-<wire x1="10.16" y1="113.03" x2="10.16" y2="128.27" width="0.1524" layer="91"/>
-<label x="10.16" y="128.27" size="1.27" layer="95" rot="R90" xref="yes"/>
-</segment>
-<segment>
 <pinref part="U$1" gate="G$1" pin="PB4/JNTRST(5T)"/>
 <wire x1="160.02" y1="45.72" x2="177.8" y2="45.72" width="0.1524" layer="91"/>
@@
 <label x="72.39" y="106.68" size="1.27" layer="95" rot="R180" xref="yes"/>
 </segment>
-</net>
+<segment>
+<pinref part="ISPJTAG" gate="A" pin="15"/>
+<wire x1="10.16" y1="113.03" x2="10.16" y2="128.27" width="0.1524" layer="91"/>
+<label x="10.16" y="128.27" size="1.27" layer="95" rot="R90" xref="yes"/>
+</segment>
+</net>
