File: zik80/schem/zik-pcb-base-bussed.sch (EAGLE design)
At the start: 37 parts, among them IC1 Z80, IC14 74LS04N

Commit message: Base PCB coming along nicely..
Parts:
- removed +3V3OUT, +5OUT, GNDOUT: (no value), pinhead:PINHD-1X3
- removed GPUHDR1: (no value), pinhead:PINHD-1X8
- removed IC2: (no value), 8Bit_Parts:AY-3-8912_28PIN
- removed IOHDR1: (no value), pinhead:PINHD-1X6
- removed ISPJTAGZDI: (no value), pinhead:PINHD-2X3
- removed LED1: (no value), SparkFun-LED:LED5MM
- removed PWRIN, PWROUT: (no value), pinhead:PINHD-1X4
- removed Q2: (no value), adafruit:CRYSTALHC49S
- removed QG1: (no value), crystal:CRYSTAL_RES-SG51
- removed R15, R16, R17, R18, R19: (no value), rcl:R-US_0204/2V
- removed RAM: AS6C1008, skeezix:DIL32
- removed U$13: PS603SPK, adafruit:PS603SPK
- removed U$9: Switch, SparkFun-Electromechanical:SWITCH-SPST-2TV
- removed U1: (no value), Zilog-eZ80-v1_0:EZ80F92AZ
- removed X4: (no value), con-yamaichi:MD06S
- removed X6: (no value), con-subd:F15HDVS
- added +3V3OUT1, +5OUT1, GNDOUT1: (no value), pinhead:PINHD-1X3
- added AY-3-8912: (no value), 8Bit_Parts:AY-3-8912_28PIN
- added BOBADDR, BOBDATA, BOBJTAG+, GPIOC-JOY0, GPIOD-JOY1: (no value), pinhead:PINHD-1X8
- added C1, C3: 22pF, rcl:C-EU025-025X050
- added C2, C4, C5, C6, C7, C9: .1uF, rcl:C-EU025-025X050
- added EZ80F93: (no value), Zilog-eZ80-v1_0:EZ80F92AZ
- added ISPZDI: (no value), pinhead:PINHD-2X3
- added JPXIN, JPXOUT: (no value), pinhead:PINHD-1X2
- added LED2: (no value), SparkFun-LED:LED5MM
- added OSCDIL14: 2.5MHz, crystal:CRYSTAL_RES-SG51
- added PS2KEYB, PWRIN1, PWROUT1, SPKR: (no value), pinhead:PINHD-1X4
- added R10, R14, R20, R21, R22, R23, R3, R6, R7, R8, R9: 10K, rcl:R-US_0204/7
- added R2: 220 O, rcl:R-US_0204/7
- added R4: 100K, rcl:R-US_0204/7
- added R5: 1K, rcl:R-US_0207/10
- added RAM-CS0: AS6C1008-55PCN, Alliance_Memory_By_element14_Batch_1:AS6C1008-55PCN
- added S1: SWITCH-MOMENTARY-2PTH, SparkFun-Electromechanical:SWITCH-MOMENTARY-2PTH
- added Z-OSC: 20Mhz, SparkFun-FreqCtrl:CRYSTALHC49US
- C10, C8: value (none) -> .1uF; device rcl:C-EU025-050X050 -> rcl:C-EU025-025X050
- R1: value 1K -> 10K; device rcl:R-US_0207/10 -> rcl:R-US_0204/7
- R11: value 2.2K -> 10K
Connections:
- removed net AT_MISO: R19.2, X6-6.F
- removed net AT_MOSI: R18.2, X6-4.F
- removed net JOYD: R16.2, X6-2.F
- removed net JOYL: R17.2, X6-3.F
- removed net JOYU: R15.2, X6-1.F
- removed net KEY_CLOCK: X4.5
- removed net KEY_DATA: X4.1
- removed net MREQ: IC1.MREQ, V1/1.B, V1/2.A
- removed net PA10: GPUHDR1.3
- removed net PA11: GPUHDR1.4
- removed net PA12: GPUHDR1.5
- removed net PA8: GPUHDR1.1
- removed net PA9: GPUHDR1.2
- removed net RD: IC1.RD, V1/1.A
- removed net SPKR: U$13.2
- removed net WR: IC1.WR, V1/2.B
- removed net XTAL1: C10.1, Q2.1
- removed net XTAL2: C8.1, Q2.2
- new net /CS0: EZ80F93.CS0, RAM-CS0.CE
- new net /CS1: EZ80F93.CS1
- new net /MEMREAD: RAM-CS0.OE, V1/2.Y
- new net /MEMWRITE: RAM-CS0.WE, V1/1.Y
- new net /MREQ: EZ80F93.MREQ, V1/1.B, V1/2.A
- new net /RD: EZ80F93.RD, V1/2.B
- new net /WR: EZ80F93.WR, V1/1.A
- new net A16: EZ80F93.A16, RAM-CS0.A16
- new net A17: EZ80F93.A17
- new net A18: EZ80F93.A18
- new net A19: EZ80F93.A19
- new net A20: EZ80F93.A20
- new net A21: EZ80F93.A21
- new net A22: EZ80F93.A22
- new net A23: EZ80F93.A23
- new net N$1: C3.1, R2.2, R4.2, Z-OSC.2
- new net N$10: AY-3-8912.CHANNEL_A, SPKR.1
- new net N$11: AY-3-8912.CLK, OSCDIL14.OUT
- new net N$12: IC1.RD
- new net N$2: LED2.A, R5.2
- new net N$6: EZ80F93.XIN, JPXIN.1
- new net N$8: AY-3-8912.CHANNEL_B, SPKR.2
- new net N$9: AY-3-8912.CHANNEL_C, SPKR.3
- new net NRST: EZ80F93.RESET, R3.1, S1.2
- new net PB0: AY-3-8912.DA0, EZ80F93.PB0/T0_IN
- new net PB1: AY-3-8912.DA1, EZ80F93.PB1/T1_IN
- new net PB2: AY-3-8912.DA2, EZ80F93.PB2/SS
- new net PB3: AY-3-8912.DA3, EZ80F93.PB3/SCK
- new net PB4: AY-3-8912.DA4, EZ80F93.PB4/T4_OUT
- new net PB5: AY-3-8912.DA5, EZ80F93.PB5/T5_OUT
- new net PC0: EZ80F93.PC0/TXD1, GPIOC-JOY0.1, R11.1
- new net PC1: EZ80F93.PC1/RXD1, GPIOC-JOY0.2, R10.1
- new net PC2: EZ80F93.PC2/RTS1, GPIOC-JOY0.3, R9.1
- new net PC3: EZ80F93.PC3/CTS1, GPIOC-JOY0.4, R8.1
- new net PC4: EZ80F93.PC4/DTR1, GPIOC-JOY0.5, R7.1
- new net PC5: AY-3-8912.BC1, EZ80F93.PC5/DSR1
- new net PC6: EZ80F93.PC6/DCD1, GPIOC-JOY0.7
- new net PC7: EZ80F93.PC7/RI1, GPIOC-JOY0.8
- new net PD0: EZ80F93.PD0/TXD0, GPIOD-JOY1.1, R23.1
- new net PD1: EZ80F93.PD1/RXD0, GPIOD-JOY1.2, R22.1
- new net PD2: EZ80F93.PD2/RTS0, GPIOD-JOY1.3, R21.1
- new net PD3: EZ80F93.PD3/CTS0, GPIOD-JOY1.4, R20.1
- new net PD4: EZ80F93.PD4/DTR0, GPIOD-JOY1.5, R14.1
- new net PD5: AY-3-8912.BDIR, EZ80F93.PD5/DSR0
- new net PD6: EZ80F93.PD6/DCD0, GPIOD-JOY1.7, PS2KEYB.4
- new net PD7: EZ80F93.PD7/RI0, GPIOD-JOY1.8, PS2KEYB.1
- new net PHI: BOBJTAG+.1, EZ80F93.PHI
- new net SCL: BOBJTAG+.7, EZ80F93.SCL
- new net SDA: BOBJTAG+.8, EZ80F93.SDA
- new net TCK_ZCL: BOBJTAG+.2, EZ80F93.TCK/ZCL, ISPZDI.4, R1.2
- new net TDI_ZDA: BOBJTAG+.4, EZ80F93.TDI/ZDA, ISPZDI.6, R6.2
- new net TDO: BOBJTAG+.5, EZ80F93.TDO
- new net TMS: BOBJTAG+.3, EZ80F93.TMS
- new net TRIGOUT: BOBJTAG+.6, EZ80F93.TRIGOUT
- new net XIN: C1.1, JPXIN.2, R4.1, Z-OSC.1
- new net XOUT: JPXOUT.1, R2.1
- net +3V3: now also +3V3OUT1.1, +3V3OUT1.2, +3V3OUT1.3, C10.1, C2.1, C4.1, C5.1, C6.1, C7.1, C8.1, C9.1, EZ80F93.+3V3@1, EZ80F93.+3V3@2, EZ80F93.+3V3@3, EZ80F93.+3V3@4, EZ80F93.+3V3@5, EZ80F93.+3V3@6, EZ80F93.+3V3@7, EZ80F93.+3V3@8, EZ80F93.WAIT, ISPZDI.1, PWRIN1.3, PWROUT1.3, R1.1, R3.2, R6.1, RAM-CS0.CE2, RAM-CS0.VCC; no longer +3V3OUT.1, +3V3OUT.2, +3V3OUT.3, PWRIN.3, PWROUT.3
- net +5V: now also +5OUT1.1, +5OUT1.2, +5OUT1.3, AY-3-8912./RESET, AY-3-8912.A8, AY-3-8912.BC2, AY-3-8912.VCC, OSCDIL14.VDD, PS2KEYB.3, PWRIN1.2, PWROUT1.2, R10.2, R11.2, R14.2, R20.2, R21.2, R22.2, R23.2, R5.1, R7.2, R8.2, R9.2; no longer +5OUT.1, +5OUT.2, +5OUT.3, PWRIN.2, PWROUT.2, R1.1
- net 5V: no longer R11.1, R15.1, R16.1, R17.1, R18.1, R19.1, X4.4
- net A0: now also BOBADDR.1, EZ80F93.A0, RAM-CS0.A0
- net A1: now also BOBADDR.2, EZ80F93.A1, RAM-CS0.A1
- net A10: now also EZ80F93.A10, RAM-CS0.A10
- net A11: now also EZ80F93.A11, RAM-CS0.A11
- net A12: now also EZ80F93.A12, RAM-CS0.A12
- net A13: now also EZ80F93.A13, RAM-CS0.A13
- net A14: now also EZ80F93.A14, RAM-CS0.A14
- net A15: now also EZ80F93.A15, RAM-CS0.A15
- net A2: now also BOBADDR.3, EZ80F93.A2, RAM-CS0.A2
- net A3: now also BOBADDR.4, EZ80F93.A3, RAM-CS0.A3
- net A4: now also BOBADDR.5, EZ80F93.A4, RAM-CS0.A4
- net A5: now also BOBADDR.6, EZ80F93.A5, RAM-CS0.A5
- net A6: now also BOBADDR.7, EZ80F93.A6, RAM-CS0.A6
- net A7: now also BOBADDR.8, EZ80F93.A7, RAM-CS0.A7
- net A8: now also EZ80F93.A8, RAM-CS0.A8
- net A9: now also EZ80F93.A9, RAM-CS0.A9
- net D0: now also BOBDATA.1, EZ80F93.D0, RAM-CS0.DQ0
- net D1: now also BOBDATA.2, EZ80F93.D1, RAM-CS0.DQ1
- net D2: now also BOBDATA.3, EZ80F93.D2, RAM-CS0.DQ2
- net D3: now also BOBDATA.4, EZ80F93.D3, RAM-CS0.DQ3
- net D4: now also BOBDATA.5, EZ80F93.D4, RAM-CS0.DQ4
- net D5: now also BOBDATA.6, EZ80F93.D5, RAM-CS0.DQ5
- net D6: now also BOBDATA.7, EZ80F93.D6, RAM-CS0.DQ6
- net D7: now also BOBDATA.8, EZ80F93.D7, RAM-CS0.DQ7
- net GND: now also AY-3-8912.VSS, C1.2, C2.2, C3.2, C4.2, C5.2, C6.2, C7.2, C9.2, EZ80F93.GND@19, EZ80F93.GND@34, EZ80F93.GND@44, EZ80F93.GND@57, EZ80F93.GND@61, EZ80F93.GND@8, EZ80F93.GND@84, EZ80F93.GND@97, GNDOUT1.1, GNDOUT1.2, GNDOUT1.3, GPIOC-JOY0.6, GPIOD-JOY1.6, ISPZDI.3, ISPZDI.5, LED2.C, OSCDIL14.VSS, PS2KEYB.2, PWRIN1.4, PWROUT1.4, RAM-CS0.VSS, S1.1, SPKR.4; no longer GNDOUT.1, GNDOUT.2, GNDOUT.3, LED1.C, PWRIN.4, PWROUT.4, U$13.1, U$9.P, X4.3, X6-8.F
- net IS_READ: no longer V1/1.Y
- net IS_WRITE: no longer V1/2.Y
- net N$3: now also EZ80F93.XOUT, JPXOUT.2; no longer LED1.A, R1.2
- net PB6: now also AY-3-8912.DA6, EZ80F93.PB6/MISO; no longer GPUHDR1.7
- net PB7: now also AY-3-8912.DA7, EZ80F93.PB7/MOSI; no longer GPUHDR1.8
- net RESETSW: no longer R11.2, U$9.O
- net VCC: now also PWRIN1.1, PWROUT1.1; no longer PWRIN.1, PWROUT.1
Other:
- note added: "- tie unused RAM addr lines to gnd - check all pull up/down and tie downs - pull up /WAIT, /RESET, etc.. check - gpu addr/data/ctrl buses - rom cart slot - drill holes - make sure connections are connected is_read/write .. ditch, use CS0/1 can't ditch is_read/write, need that for OE/WE .. pull up/downs needed on CS, resets, etc? - NMI to user switch to gnd? - rev2: IOREQ, handle OUT for something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"
- note added: "Note that GPIO C and D have serial on them; instead of 2nd joystick, use it for serial debugging, forex. Just don't populate the pullup resistors in that case or serial fail."
- note added: "joy up joy down joy left joy right joy fire GND ps2 clk ps2 data"
- note added: "joy up joy down joy left joy right joy fire GND vblank in frame rdy out"
- note removed: "AT_CLOCK"
- note removed: "Atari Joystick"
- note removed: "Button"
- note removed: "Down"
- note removed: "Left"
- note removed: "Legend: + usart1 video + i2c p1: usart CK p2: TX p3: RX p4: CTS p5: RTS p6: p7: i2c scl p8: i2c sda"
- note removed: "Legend: p1: Console TX (send from micro): usart2 p2: Console RX (receive to micro): usart2 p3: p4: p5: p6: vblank"
- note removed: "PIAZ. SPKR"
- note removed: "PS/2 Keyb"
- note removed: "Reset Switch - RESET must hold for >3 clock cycles"
- note removed: "Right"
- note removed: "Up"
- note removed: "Zilog ISP header? Z-debug header for own programmer/debug? OCI (jtag support?!) AY-3-8910 .. shift reg from z80? vblank and frameready where?"
- note removed: "eZ80 24 GPIO: - 10 (8d, 2 ctrl) for AY-3-8912 - 1 vblank in - 1 frame ready out - 2 ps2 keyb - 5 = joy4+1 - 5 = joy4+1 == 24 used"
- moved on the sheet: ADDRESS_BUS, C10, C8, CTRL_BUS, DATA_BUS, R1, R11, V1/1, V1/2

Commit message: base pcb with built in ez80 is more or less ready; time to make pcb..
Parts:
- removed AT28C256-ROM: AT28C256, skeezix:AT28C256
- removed IC1: Z80, zilog:Z80CPU
- removed IC14: 74LS04N, 74xx-us:74LS04N
- removed SRAM-128K: CY7C1019CV33-10ZXC, memory-sram:CY7C1019CV33-10ZXC
- added 74HCT04: 74LS04N, 74xx-us:74LS04N
- added BOBMISC: (no value), pinhead:PINHD-1X8
- added CART-CS1: ZIKCART36, skeezix:ZIKCART36
- renumbered +3V3OUT1 to +3V3OUT, +5OUT1 to +5OUT, AY-3-8912 to AY-3-8912-CS2, GNDOUT1 to GNDOUT
Connections:
- removed net 5V: AT28C256-ROM.VCC, IC1.VCC, R12.2, R13.2, SRAM-128K.+3V@1, SRAM-128K.+3V@2
- removed net CPUWANTINT: R13.1
- removed net IOREQINT: IC1.IORQ
- removed net IS_RAM: AT28C256-ROM./CE, IC14A.I, V1/3.Y
- removed net IS_READ: AT28C256-ROM./OE, SRAM-128K.OE
- removed net IS_WRITE: SRAM-128K.WE
- removed net N$12: IC1.RD
- removed net N$4: IC1.BUSRQ, IC1.NMI, IC1.WAIT, R12.1
- removed net N$7: IC14A.O, SRAM-128K.CE
- removed net OPFETCH: IC1.M1
- removed net RESETSW: IC1.RESET
- removed net Z_CLK: IC1.CLK
- new net +CS2: 74HCT04A.O, AY-3-8912-CS2.A8
- new net +MEMWRITE: 74HCT04B.O, AY-3-8912-CS2.BDIR
- new net /BUSACK: CTRL_BUS.15, CTRL_BUS.16, EZ80F93.BUSACK
- new net /BUSREQ: CTRL_BUS.13, CTRL_BUS.14, EZ80F93.BUSREQ
- new net /CS2: 74HCT04A.I, CTRL_BUS.10, CTRL_BUS.9, EZ80F93.CS2
- new net /IOREQ: BOBMISC.4, EZ80F93.IORQ, R13.2
- new net HALT_SLP: BOBMISC.2, EZ80F93.HALT_SLP
- new net NMI: BOBMISC.1, EZ80F93.NMI, R12.2
- new net RTC_VDD: BOBMISC.6, EZ80F93.RTC_VDD
- new net RTC_XIN: BOBMISC.8, EZ80F93.RTC_XIN
- new net RTC_XOUT: BOBMISC.7, EZ80F93.RTC_XOUT
- net +3V3: now also CART-CS1.VCC33, R12.1, R13.1
- net +5V: now also CART-CS1.VCC5; no longer AY-3-8912-CS2.A8
- net /CS0: now also CTRL_BUS.5, CTRL_BUS.6
- net /CS1: now also CART-CS1./CE, CTRL_BUS.7, CTRL_BUS.8
- net /MEMREAD: now also CART-CS1./OE, CTRL_BUS.1, CTRL_BUS.2
- net /MEMWRITE: now also 74HCT04B.I, CART-CS1./WE, CTRL_BUS.3, CTRL_BUS.4
- net /MREQ: now also CTRL_BUS.11, CTRL_BUS.12
- net A0: now also ADDRESS_BUS.1, AY-3-8912-CS2.BC1, CART-CS1.A0; no longer AT28C256-ROM.A0, IC1.A0, SRAM-128K.A0
- net A1: now also ADDRESS_BUS.2, CART-CS1.A1; no longer AT28C256-ROM.A1, IC1.A1, SRAM-128K.A1
- net A10: now also ADDRESS_BUS.11, CART-CS1.A10; no longer AT28C256-ROM.A10, IC1.A10, SRAM-128K.A10
- net A11: now also ADDRESS_BUS.12, CART-CS1.A11; no longer AT28C256-ROM.A11, IC1.A11, SRAM-128K.A11
- net A12: now also ADDRESS_BUS.13, CART-CS1.A12; no longer AT28C256-ROM.A12, SRAM-128K.A12
- net A13: now also ADDRESS_BUS.14, CART-CS1.A13; no longer AT28C256-ROM.A13, SRAM-128K.A13
- net A14: now also ADDRESS_BUS.15, CART-CS1.A14; no longer AT28C256-ROM.A14, IC1.A14, SRAM-128K.A14, V1/3.A
- net A15: now also ADDRESS_BUS.16, CART-CS1.A15; no longer IC1.A15, SRAM-128K.A15, V1/3.B
- net A16: now also ADDRESS_BUS.17, CART-CS1.A16
- net A17: now also ADDRESS_BUS.18, CART-CS1.A17
- net A18: now also ADDRESS_BUS.19, CART-CS1.A18
- net A19: now also ADDRESS_BUS.20, CART-CS1.A19
- net A2: now also ADDRESS_BUS.3, CART-CS1.A2; no longer AT28C256-ROM.A2, IC1.A2, SRAM-128K.A2
- net A20: now also ADDRESS_BUS.21, CART-CS1.A20
- net A21: now also ADDRESS_BUS.22, CART-CS1.A21
- net A3: now also ADDRESS_BUS.4, CART-CS1.A3; no longer AT28C256-ROM.A3, IC1.A3, SRAM-128K.A3
- net A4: now also ADDRESS_BUS.5, CART-CS1.A4; no longer AT28C256-ROM.A4, IC1.A4, SRAM-128K.A4
- net A5: now also ADDRESS_BUS.6, CART-CS1.A5; no longer AT28C256-ROM.A5, IC1.A5, SRAM-128K.A5
- net A6: now also ADDRESS_BUS.7, CART-CS1.A6; no longer AT28C256-ROM.A6, IC1.A6, SRAM-128K.A6
- net A7: now also ADDRESS_BUS.8, CART-CS1.A7; no longer AT28C256-ROM.A7, IC1.A7, SRAM-128K.A7
- net A8: now also ADDRESS_BUS.9, CART-CS1.A8; no longer AT28C256-ROM.A8, IC1.A8, SRAM-128K.A8
- net A9: now also ADDRESS_BUS.10, CART-CS1.A9; no longer AT28C256-ROM.A9, IC1.A9, SRAM-128K.A9
- net D0: now also AY-3-8912-CS2.DA0, CART-CS1.D0, DATA_BUS.1; no longer AT28C256-ROM.IO0, IC1.D0, SRAM-128K.I/O00
- net D1: now also AY-3-8912-CS2.DA1, CART-CS1.D1, DATA_BUS.2; no longer AT28C256-ROM.IO1, IC1.D1, SRAM-128K.I/O01
- net D2: now also AY-3-8912-CS2.DA2, CART-CS1.D2, DATA_BUS.3; no longer AT28C256-ROM.IO2, IC1.D2, SRAM-128K.I/O02
- net D3: now also AY-3-8912-CS2.DA3, CART-CS1.D3, DATA_BUS.4; no longer AT28C256-ROM.IO3, IC1.D3, SRAM-128K.I/O03
- net D4: now also AY-3-8912-CS2.DA4, CART-CS1.D4, DATA_BUS.5; no longer AT28C256-ROM.IO4, IC1.D4, SRAM-128K.I/O04
- net D5: now also AY-3-8912-CS2.DA5, CART-CS1.D5, DATA_BUS.6; no longer AT28C256-ROM.IO5, IC1.D5, SRAM-128K.I/O05
- net D6: now also AY-3-8912-CS2.DA6, CART-CS1.D6, DATA_BUS.7; no longer AT28C256-ROM.IO6, IC1.D6, SRAM-128K.I/O06
- net D7: now also AY-3-8912-CS2.DA7, CART-CS1.D7, DATA_BUS.8; no longer AT28C256-ROM.IO7, IC1.D7, SRAM-128K.I/O07
- net GND: now also CART-CS1.GND; no longer AT28C256-ROM.GND, GPIOC-JOY0.6, GPIOD-JOY1.6, IC1.GND, SRAM-128K.A16, SRAM-128K.GND@1, SRAM-128K.GND@2
- net PB0: no longer AY-3-8912-CS2.DA0
- net PB1: no longer AY-3-8912-CS2.DA1
- net PB2: no longer AY-3-8912-CS2.DA2
- net PB3: no longer AY-3-8912-CS2.DA3
- net PB4: no longer AY-3-8912-CS2.DA4
- net PB5: no longer AY-3-8912-CS2.DA5
- net PB6: no longer AY-3-8912-CS2.DA6
- net PB7: no longer AY-3-8912-CS2.DA7
- net PC5: now also GPIOC-JOY0.6; no longer AY-3-8912-CS2.BC1
- net PD5: now also GPIOD-JOY1.6; no longer AY-3-8912-CS2.BDIR
- net PHI: now also BOBMISC.3; no longer BOBJTAG+.1
- net TCK_ZCL: now also BOBJTAG+.1; no longer BOBJTAG+.2
- net TDI_ZDA: now also BOBJTAG+.3; no longer BOBJTAG+.4
- net TDO: now also BOBJTAG+.4; no longer BOBJTAG+.5
- net TMS: now also BOBJTAG+.2; no longer BOBJTAG+.3
- net TRIGOUT: now also BOBJTAG+.5; no longer BOBJTAG+.6
Other:
- note added: "- drill holes - identification stamp - GPIO PB unused - rev2: IOREQ, handle OUT for something/BoB? - rev2: amplifier 2n2222 as per http below? mix all 3 channels together to another pin on speaker header? amp on board? - rev2: ?? put PSG back onto GPIO PB, drop the inverters, use GPIO for A8 and BDIR and BC1? Bus idea here: http://z80.hit.bg/z80/eZ80.pdf - rev2: zikcart - tie unused addr to gnd?"
- note added: "Assignments: GPIO PB: unused GPIO PC: 6 for joy1 2 for vbl/frameready GPIO PD: 6 for joy-2 2 for keyb"
- note added: "No need for Chip Select lines on ctrl-bus from GPU, since eZ80 will maintain Chip Select lines during BUSACK period. - put them anyway, even though gpu doesn't use them, in case we want to manually do them from other guys GPIO say.."
- note added: "joy up joy down joy left joy right joy fire joy fire2 or unused vblank in frame rdy out"
- note added: "joy up joy down joy left joy right joy fire2/unused GND ps2 clk ps2 data"
- note removed: "- tie unused RAM addr lines to gnd - check all pull up/down and tie downs - pull up /WAIT, /RESET, etc.. check - gpu addr/data/ctrl buses - rom cart slot - drill holes - make sure connections are connected is_read/write .. ditch, use CS0/1 can't ditch is_read/write, need that for OE/WE .. pull up/downs needed on CS, resets, etc? - NMI to user switch to gnd? - rev2: IOREQ, handle OUT for something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"
- note removed: "/"
- note removed: "joy up joy down joy left joy right joy fire GND ps2 clk ps2 data"
- note removed: "joy up joy down joy left joy right joy fire GND vblank in frame rdy out"
- moved on the sheet: ADDRESS_BUS, CTRL_BUS, DATA_BUS, R12, R13

Commit message: Working on base pcb .. nearly there, but last few traces will take hours..
Parts:
- removed 74HCT04: 74LS04N, 74xx-us:74LS04N
- removed BOBADDR, BOBDATA: (no value), pinhead:PINHD-1X8
- removed JPXIN, JPXOUT: (no value), pinhead:PINHD-1X2
- removed V1: 7432N, 74ttl-din:7432N
- added BOBGPIOB: (no value), pinhead:PINHD-1X8
- added BOBI2C: (no value), pinhead:PINHD-1X2
- added IC1: 7432N, 74xx-us-33v-skeezix:7432N
- added IC2: 7404N, 74xx-us-5v-skeezix:7404N
Connections:
- removed net N$3: EZ80F93.XOUT, JPXOUT.2
- removed net N$6: EZ80F93.XIN, JPXIN.1
- new net /CS3: BOBMISC.5, EZ80F93.CS3
- net +CS2: now also IC2A.O; no longer 74HCT04A.O
- net +MEMWRITE: now also IC2B.O; no longer 74HCT04B.O
- net /CS2: now also IC2A.I; no longer 74HCT04A.I
- net /MEMREAD: now also IC1B.O; no longer V1/2.Y
- net /MEMWRITE: now also IC1A.O, IC2B.I; no longer 74HCT04B.I, V1/1.Y
- net /MREQ: now also IC1A.I1, IC1B.I0; no longer V1/1.B, V1/2.A
- net /RD: now also IC1B.I1; no longer V1/2.B
- net /WR: now also IC1A.I0; no longer V1/1.A
- net A0: no longer BOBADDR.1
- net A1: no longer BOBADDR.2
- net A2: no longer BOBADDR.3
- net A3: no longer BOBADDR.4
- net A4: no longer BOBADDR.5
- net A5: no longer BOBADDR.6
- net A6: no longer BOBADDR.7
- net A7: no longer BOBADDR.8
- net D0: no longer BOBDATA.1
- net D1: no longer BOBDATA.2
- net D2: no longer BOBDATA.3
- net D3: no longer BOBDATA.4
- net D4: no longer BOBDATA.5
- net D5: no longer BOBDATA.6
- net D6: no longer BOBDATA.7
- net D7: no longer BOBDATA.8
- net GND: now also IC1C.I0, IC1C.I1, IC1D.I0, IC1D.I1, IC2C.I, IC2D.I, IC2E.I, IC2F.I
- net PB0: now also BOBGPIOB.1
- net PB1: now also BOBGPIOB.2
- net PB2: now also BOBGPIOB.3
- net PB3: now also BOBGPIOB.4
- net PB4: now also BOBGPIOB.5
- net PB5: now also BOBGPIOB.6
- net PB6: now also BOBGPIOB.7
- net PB7: now also BOBGPIOB.8
- net SCL: now also BOBI2C.1; no longer BOBJTAG+.7
- net SDA: now also BOBI2C.2; no longer BOBJTAG+.8
- net XIN: now also EZ80F93.XIN; no longer JPXIN.2
- net XOUT: now also EZ80F93.XOUT; no longer JPXOUT.1
Other:
- note added: "- brd positions - drill holes - identification stamp - Big Question: V-in-low and V-in-high from eZ80 to 74HC32-at-3.3 are close --> could bodge 5v into 73LS32 and it should work - GPIO PB unused -> sent to BoB for LEDs/switches - rev2: IOREQ, handle OUT for something/BoB? - rev2: amplifier 2n2222 as per http below? mix all 3 channels together to another pin on speaker header? amp on board? - rev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"
- note added: "Jeff Mitchell 2014 www.zikzak.ca"
- note removed: "- drill holes - identification stamp - GPIO PB unused - rev2: IOREQ, handle OUT for something/BoB? - rev2: amplifier 2n2222 as per http below? mix all 3 channels together to another pin on speaker header? amp on board? - rev2: ?? put PSG back onto GPIO PB, drop the inverters, use GPIO for A8 and BDIR and BC1? Bus idea here: http://z80.hit.bg/z80/eZ80.pdf - rev2: zikcart - tie unused addr to gnd?"
