File: zik80/schem/zik-pcb-sbc-ez80stm100p.sch (EAGLE design)
At the start: 96 parts, among them IC1 7432N, IC2 7404N

Commit message: working on first cut of new pcb layout
Parts:
- R16: value (none) -> 2K
- R17: value (none) -> 1K
Connections:
- removed net PB3: ISPJTAG.13
- new net ZNRST: EZ80F93.RESET, ISPJTAG.15, R3.1, S1.2
- net /CS1: now also ISPJTAG.13
- net GND: now also BOBJTAG+.6
- net NRST: no longer EZ80F93.RESET, ISPJTAG.15, R3.1, S1.2
Changed lines of the file:
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@@
 <setting verticaltext="up"/>
 </settings>
-<grid distance="0.05" unitdist="inch" unit="inch" style="dots" multiple="1" display="yes" altdistance="0.01" altunitdist="inch" altunit="inch"/>
+<grid distance="0.1" unitdist="inch" unit="inch" style="lines" multiple="1" display="no" altdistance="0.01" altunitdist="inch" altunit="inch"/>
 <layers>
 <layer number="1" name="Top" color="4" fill="1" visible="no" active="no"/>
@@
 <part name="GND33" library="supply1" deviceset="GND" device=""/>
 <part name="VGAHDR" library="pinhead" deviceset="PINHD-1X6" device=""/>
-<part name="R16" library="rcl" deviceset="R-US_" device="0207/10"/>
-<part name="R17" library="rcl" deviceset="R-US_" device="0207/10"/>
+<part name="R16" library="rcl" deviceset="R-US_" device="0207/10" value="2K"/>
+<part name="R17" library="rcl" deviceset="R-US_" device="0207/10" value="1K"/>
 <part name="R18" library="rcl" deviceset="R-US_" device="0207/10"/>
 <part name="R19" library="rcl" deviceset="R-US_" device="0207/10"/>
@@
 </segment>
 <segment>
-<wire x1="180.34" y1="250.19" x2="185.42" y2="250.19" width="0.1524" layer="91"/>
+<wire x1="179.07" y1="250.19" x2="185.42" y2="250.19" width="0.1524" layer="91"/>
 <label x="185.42" y="250.19" size="1.27" layer="95" xref="yes"/>
+<pinref part="BOBJTAG+" gate="A" pin="6"/>
 </segment>
 <segment>
@@
 <label x="1085.85" y="109.22" size="1.27" layer="95" rot="R180" xref="yes"/>
 <pinref part="STM32F4" gate="G$1" pin="VSS_3"/>
-<wire x1="1092.2" y1="114.3" x2="1085.85" y2="114.3" width="0.1524" layer="91"/>
-<label x="1085.85" y="114.3" size="1.27" layer="95" rot="R180" xref="yes"/>
-<pinref part="STM32F4" gate="G$1" pin="VSS_1"/>
 </segment>
 <segment>
@@
 <label x="1078.23" y="106.68" size="1.27" layer="95" rot="R180" xref="yes"/>
 <pinref part="STM32F4" gate="G$1" pin="VSS_4"/>
-<wire x1="1092.2" y1="111.76" x2="1078.23" y2="111.76" width="0.1524" layer="91"/>
-<label x="1078.23" y="111.76" size="1.27" layer="95" rot="R180" xref="yes"/>
-<pinref part="STM32F4" gate="G$1" pin="VSS_2"/>
 </segment>
 <segment>
@@
 <wire x1="1019.81" y1="104.14" x2="1019.81" y2="105.41" width="0.1524" layer="91"/>
 </segment>
+<segment>
+<pinref part="STM32F4" gate="G$1" pin="VSS_1"/>
+<wire x1="1092.2" y1="114.3" x2="1085.85" y2="114.3" width="0.1524" layer="91"/>
+<label x="1085.85" y="114.3" size="1.27" layer="95" rot="R180" xref="yes"/>
+</segment>
+<segment>
+<pinref part="STM32F4" gate="G$1" pin="VSS_2"/>
+<wire x1="1092.2" y1="111.76" x2="1078.23" y2="111.76" width="0.1524" layer="91"/>
+<label x="1078.23" y="111.76" size="1.27" layer="95" rot="R180" xref="yes"/>
+</segment>
 </net>
 <net name="PB6" class="0">
@@
 </segment>
 <segment>
-<wire x1="426.72" y1="143.51" x2="425.45" y2="143.51" width="0.1524" layer="91"/>
 <label x="417.83" y="143.51" size="1.27" layer="95" rot="R180" xref="yes"/>
 <pinref part="BOBADDR" gate="A" pin="1"/>
 <wire x1="425.45" y1="143.51" x2="417.83" y2="143.51" width="0.1524" layer="91"/>
-<junction x="425.45" y="143.51"/>
 </segment>
 </net>
@@
 </segment>
 </net>
-<net name="NRST" class="0">
+<net name="ZNRST" class="0">
 <segment>
 <pinref part="S1" gate="G$1" pin="2"/>
@@
 <junction x="43.18" y="85.09"/>
 <pinref part="EZ80F93" gate="G$1" pin="RESET"/>
-</segment>
-<segment>
-<wire x1="1170.94" y1="17.78" x2="1174.75" y2="17.78" width="0.1524" layer="91"/>
-<label x="1177.29" y="17.78" size="1.27" layer="95" rot="MR180" xref="yes"/>
-<pinref part="S2" gate="G$1" pin="2"/>
-<wire x1="1174.75" y1="17.78" x2="1177.29" y2="17.78" width="0.1524" layer="91"/>
-<wire x1="1174.75" y1="3.81" x2="1174.75" y2="17.78" width="0.1524" layer="91"/>
-<junction x="1174.75" y="17.78"/>
-<pinref part="STM32F4" gate="G$1" pin="NRST"/>
+<label x="50.8" y="85.09" size="1.27" layer="95" rot="R270" xref="yes"/>
 </segment>
 <segment>
@@
 <wire x1="1037.59" y1="121.92" x2="1037.59" y2="129.54" width="0.1524" layer="91"/>
 <wire x1="1037.59" y1="129.54" x2="1092.2" y2="129.54" width="0.1524" layer="91"/>
-<wire x1="1035.05" y1="121.92" x2="1037.59" y2="121.92" width="0.1524" layer="91"/>
+<wire x1="1033.78" y1="121.92" x2="1037.59" y2="121.92" width="0.1524" layer="91"/>
 <junction x="1037.59" y="121.92"/>
-<label x="1035.05" y="121.92" size="1.27" layer="95" rot="R270" xref="yes"/>
+<label x="1033.78" y="121.92" size="1.27" layer="95" rot="R270" xref="yes"/>
 </segment>
 <segment>
@@
 </segment>
 </net>
-<net name="PB3" class="0">
-<segment>
-<pinref part="ISPJTAG" gate="A" pin="13"/>
-<wire x1="1012.19" y1="242.57" x2="1012.19" y2="250.19" width="0.1524" layer="91"/>
-<label x="1012.19" y="250.19" size="1.27" layer="95" rot="R90" xref="yes"/>
-</segment>
-</net>
 <net name="PC0" class="0">
 <segment>
@@
 <label x="1076.96" y="48.26" size="1.27" layer="95" rot="R180" xref="yes"/>
 </segment>
+<segment>
+<pinref part="ISPJTAG" gate="A" pin="13"/>
+<wire x1="1012.19" y1="242.57" x2="1012.19" y2="250.19" width="0.1524" layer="91"/>
+<label x="1012.19" y="250.19" size="1.27" layer="95" rot="R90" xref="yes"/>
+</segment>
 </net>
 <net name="A16" class="0">
@@
 </segment>
 </net>
+<net name="NRST" class="0">
+<segment>
+<wire x1="1170.94" y1="17.78" x2="1174.75" y2="17.78" width="0.1524" layer="91"/>
+<label x="1177.29" y="17.78" size="1.27" layer="95" rot="MR180" xref="yes"/>
+<pinref part="S2" gate="G$1" pin="2"/>
+<wire x1="1174.75" y1="17.78" x2="1177.29" y2="17.78" width="0.1524" layer="91"/>
+<wire x1="1174.75" y1="3.81" x2="1174.75" y2="17.78" width="0.1524" layer="91"/>
+<junction x="1174.75" y="17.78"/>
+<pinref part="STM32F4" gate="G$1" pin="NRST"/>
+</segment>
+</net>

Commit message: Fiddling with sbc board layout
Connections:
- net NRST: now also ISPJTAG.15
- net ZNRST: no longer ISPJTAG.15
Other:
- moved on the sheet: BOB-PA, C11, C12, C13, C14, C15, C16, C17, C18, C19, C20, C21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

Commit message: SBC pcb design rev2, sprite demo on ARM
Parts:
- removed AY-3-8912-CS2: (no value), 8Bit_Parts:AY-3-8912_28PIN
- added AY-3-8913-CS2: (no value), 8Bit_Parts:AY-3-8912_24PIN-6
Connections:
- removed net N$10: AY-3-8912-CS2.CHANNEL_A, SPKR.1
- removed net N$8: AY-3-8912-CS2.CHANNEL_B, SPKR.2
- removed net N$9: AY-3-8912-CS2.CHANNEL_C, SPKR.3
- new net N$26: AY-3-8913-CS2.CHANNEL_A, SPKR.1
- new net N$27: AY-3-8913-CS2.CHANNEL_B, SPKR.2
- new net N$28: AY-3-8913-CS2.CHANNEL_C, SPKR.3
- net +5V: now also AY-3-8913-CS2./RESET, AY-3-8913-CS2.A8, AY-3-8913-CS2.VCC; no longer AY-3-8912-CS2./RESET, AY-3-8912-CS2.BC2, AY-3-8912-CS2.VCC
- net +CS2: no longer AY-3-8912-CS2.A8
- net +MEMWRITE: now also AY-3-8913-CS2.BDIR; no longer AY-3-8912-CS2.BDIR
- net /CS2: now also AY-3-8913-CS2./CS
- net A0: now also AY-3-8913-CS2.BC1; no longer AY-3-8912-CS2.BC1
- net D0: now also AY-3-8913-CS2.DA0; no longer AY-3-8912-CS2.DA0
- net D1: now also AY-3-8913-CS2.DA1; no longer AY-3-8912-CS2.DA1
- net D2: now also AY-3-8913-CS2.DA2; no longer AY-3-8912-CS2.DA2
- net D3: now also AY-3-8913-CS2.DA3; no longer AY-3-8912-CS2.DA3
- net D4: now also AY-3-8913-CS2.DA4; no longer AY-3-8912-CS2.DA4
- net D5: now also AY-3-8913-CS2.DA5; no longer AY-3-8912-CS2.DA5
- net D6: now also AY-3-8913-CS2.DA6; no longer AY-3-8912-CS2.DA6
- net D7: now also AY-3-8913-CS2.DA7; no longer AY-3-8912-CS2.DA7
- net GND: now also AY-3-8913-CS2./A9, AY-3-8913-CS2.VSS, AY-3-8913-CS2.VSS2; no longer AY-3-8912-CS2.VSS
- net N$11: now also AY-3-8913-CS2.CLK; no longer AY-3-8912-CS2.CLK
Other:
- note added: "- OOPS: ay-3-8912 not really suitable here, since the A8/A9 mechanism doesn't high-Z; we need -8913 variant with true /CS - keep all bus breakout pins? or keep less so, and open up IOreq for expansion? what about stm32 breakout? REV2++: Bigger drill holes for cart edge conn .. also check spacing? ++ split off addr to 16+6 connectors ++ CHG edge connector to side mount with pads, instead of drill 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"
- note removed: "- keep all bus breakout pins? or keep less so, and open up IOreq for expansion? what about stm32 breakout? REV2++: Bigger drill holes for cart edge conn .. also check spacing? ++ split off addr to 16+6 connectors ++ CHG edge connector to side mount with pads, instead of drill holes at all; just squish the pins or pads and solder! ++ Clear space around audio osc .. esp resistor needs to move - Big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"
- moved on the sheet: OSCDIL14, SPKR

Commit message: schem exported image
Other:
- note added: "Zikzak SBC - Single board computer Jeff Mitchell 2014"
- note removed: "- OOPS: ay-3-8912 not really suitable here, since the A8/A9 mechanism doesn't high-Z; we need -8913 variant with true /CS - keep all bus breakout pins? or keep less so, and open up IOreq for expansion? what about stm32 breakout? REV2++: Bigger drill holes for cart edge conn .. also check spacing? ++ split off addr to 16+6 connectors ++ CHG edge connector to side mount with pads, instead of drill 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"
Changed lines of the file:
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@@
 <setting verticaltext="up"/>
 </settings>
-<grid distance="0.05" unitdist="inch" unit="inch" style="dots" multiple="1" display="yes" altdistance="0.01" altunitdist="inch" altunit="inch"/>
+<grid distance="0.1" unitdist="inch" unit="inch" style="lines" multiple="1" display="no" altdistance="0.01" altunitdist="inch" altunit="inch"/>
 <layers>
 <layer number="1" name="Top" color="4" fill="1" visible="no" active="no"/>
@@
 <plain>
 <rectangle x1="21.59" y1="-207.518" x2="100.584" y2="-190.5" layer="206"/>
-<text x="222.25" y="-86.36" size="5.08" layer="91">- OOPS: ay-3-8912 not really suitable here, since the A8/A9 mechanism doesn't high-Z; we need -8913 variant with true /CS
-- keep all bus breakout pins? or keep less so, and open up IOreq for expansion? what about stm32 breakout?
-REV2++: Bigger drill holes for cart edge conn .. also check spacing?
-++ split off addr to 16+6 connectors
-++ CHG edge connector to side mount with pads, instead of drill holes at all; just squish the pins or pads and solder!
-++ Clear space around audio osc .. esp resistor needs to move
-- Big Question: V-in-low and V-in-high from eZ80 to 74HC32-at-3.3 are close
---&gt; could bodge 5v into 73LS32 and it should work
-- GPIO PB unused -&gt; sent to BoB for LEDs/switches
-- rev2: IOREQ, handle OUT for something/BoB?
-- rev2: amplifier 2n2222 as per http below? mix all 3 channels together to another pin on speaker header? amp on board?
-- rev2: ?? put PSG back onto GPIO PB, drop the inverters, use GPIO for A8 and BDIR and BC1? Bus idea here: http://z80.hit.bg/z80/eZ80.pdf
-- rev2: zikcart - tie unused addr to gnd?
-- rev2: change ctrl bus, add /cs3 for gpu.. bus to gpu, sweet</text>
 <text x="40.64" y="311.15" size="1.778" layer="94">Power-In header
 - VCC
@@
 PA8-2 - usart1
 --&gt; could jumper to eZ80 GPIO/serial</text>
-<text x="215.9" y="-168.91" size="5.08" layer="91">Of interest..
+<text x="330.2" y="-29.21" size="5.08" layer="91">Of interest..
 - Bus expansion:
   -&gt; /CS3 is on Breakout pins too, not just to gpu
@@
 - SD card .. see GPIO B, wide open SPI :)
 - ethernet .. not direct, thats eZ80F91, not F93; perhaps an i2c, SPI, serial, or bus addition ethernet or wifi...</text>
+<text x="330.2" y="55.88" size="6.4516" layer="91">Zikzak SBC - Single board computer
+Jeff Mitchell 2014</text>
 </plain>
 <instances>
