File: zik80/schem/zok-atmega644-bob.sch (EAGLE design)
At the start: 45 parts, among them IC1 TPS7133QP, U2 FT232RLSSOP

Commit message: Finished up zok atmega bob rev1, and zikzak sbc rev3
Parts:
- removed C10, C9: 22pf, rcl:C-EU025-050X050
- removed C8: (no value), rcl:C-EU025-050X050
- removed LED1, LED2: (no value), led:LEDMINI-TOP
- removed POWER-CLOCK: (no value), pinhead:PINHD-1X8
- removed R7: (no value), rcl:R-US_0204/2V
- added ALWAYS-ON, PD0-TXD, PD1-RXD: (no value), pinhead:PINHD-1X2
- added C4, C5: .1uF, rcl:C-EU025-025X050
- added C6: 22pF, rcl:C-EU025-025X050
- added OPTLED1, OPTLED2: (no value), SparkFun-LED:LED5MM
- added P1, P10, P100, P101, P102, P103, P104, P105, P106, P107, P108, P109, P11, P110, P111, P112, P113, P114, P115, P116, P117, P118, P119, P12, P120, P121, P122, P123, P124, P125, P126, P127, P128, P129, P13, P130, P139, P14, P140, P141, P142, P143, P144, P145, P146, P147, P148, P149, P15, P150, P151, P152, P153, P154, P155, P156, P157, P158, P159, P16, P160, P161, P162, P163, P164, P165, P166, P167, P168, P169, P17, P170, P171, P172, P173, P174, P175, P176, P177, P178, P179, P18, P180, P183, P184, P185, P186, P187, P188, P189, P19, P190, P191, P192, P193, P194, P195, P196, P197, P198, P199, P2, P20, P200, P201, P202, P203, P204, P205, P206, P207, P208, P21, P211, P212, P213, P214, P215, P216, P217, P218, P219, P22, P220, P221, P222, P223, P224, P225, P226, P227, P228, P229, P23, P230, P231, P232, P233, P234, P235, P236, P237, P238, P239, P24, P240, P241, P242, P243, P244, P245, P246, P247, P248, P249, P25, P250, P251, P252, P253, P254, P255, P256, P257, P258, P259, P26, P260, P261, P262, P263, P264, P265, P266, P267, P268, P269, P27, P270, P271, P272, P273, P274, P275, P276, P277, P278, P279, P28, P280, P281, P282, P283, P284, P285, P286, P287, P288, P289, P29, P290, P291, P292, P293, P294, P295, P296, P297, P298, P299, P3, P30, P300, P301, P302, P303, P304, P305, P306, P307, P308, P309, P31, P310, P311, P312, P313, P314, P315, P316, P317, P318, P319, P32, P320, P321, P322, P323, P324, P325, P326, P327, P328, P329, P33, P330, P331, P332, P333, P334, P335, P336, P337, P338, P339, P34, P340, P341, P342, P343, P344, P345, P346, P347, P348, P349, P35, P350, P351, P352, P353, P354, P355, P356, P357, P358, P359, P36, P360, P361, P362, P363, P364, P365, P366, P367, P368, P369, P37, P370, P371, P372, P373, P374, P375, P376, P377, P378, P379, P38, P380, P381, P382, P383, P384, P385, P386, P387, P388, P389, P39, P390, P391, P392, P393, P394, P395, P396, P397, P398, P399, P4, P40, P400, P401, P402, P403, P404, P405, P406, P407, P408, P409, P41, P410, P411, P412, P42, P43, P44, P45, P46, P47, P48, P49, P5, P50, P51, P52, P53, P54, P55, P56, P57, P58, P59, P6, P60, P61, P62, P63, P64, P65, P66, P67, P68, P69, P7, P70, P71, P72, P73, P74, P75, P76, P77, P78, P79, P8, P80, P81, P82, P83, P84, P85, P86, P87, P88, P89, P9, P90, P91, P92, P93, P94, P95, P96, P97, P98, P99: (no value), wirepad:1,6/0,9
- added R8: 10K, rcl:R-US_0204/7
- C1, C2: value 0.1uF -> .1uF; device SparkFun:CAP0402-CAP -> rcl:C-EU025-025X050
- C7: value (none) -> 22pF; device rcl:C-EU025-050X050 -> rcl:C-EU025-025X050
- R1: device rcl:R-US_0207/10 -> rcl:R-US_0204/7
- R2, R3, R6: value (none) -> 330 ohm; device rcl:R-US_0204/2V -> rcl:R-US_0204/7
- R4: device rcl:R-US_0204/2V -> rcl:R-US_0204/7
- R5: value 10K -> 330 ohm; device rcl:R-US_0204/2V -> rcl:R-US_0204/7
- RXLED, TXLED: device led:LEDMINI-TOP -> SparkFun-LED:LED5MM
Connections:
- new net N$12: PD0-TXD.1, U2.TXD
- new net N$13: PD1-RXD.1, U2.RXD
- net +5V: now also ALWAYS-ON.2
- net AREF: no longer POWER-CLOCK.8
- net AT_RESET: no longer POWER-CLOCK.1
- net GND: now also C4.2, C5.2, C6.2, OPTLED1.C, OPTLED2.C, P1.P, P10.P, P11.P, P12.P, P13.P, P14.P, P15.P, P16.P, P17.P, P18.P, P183.P, P184.P, P185.P, P186.P, P187.P, P188.P, P189.P, P19.P, P190.P, P191.P, P192.P, P193.P, P194.P, P195.P, P196.P, P197.P, P198.P, P199.P, P2.P, P20.P, P200.P, P201.P, P202.P, P203.P, P204.P, P205.P, P206.P, P207.P, P208.P, P21.P, P22.P, P23.P, P24.P, P25.P, P26.P, P27.P, P28.P, P29.P, P3.P, P30.P, P31.P, P32.P, P33.P, P34.P, P35.P, P36.P, P4.P, P5.P, P6.P, P7.P, P8.P, P9.P; no longer C10.2, C8.2, C9.2, LED1.C, LED2.C, POWER-CLOCK.3, POWER-CLOCK.7
- net N$1: now also R8.1; no longer R4.2
- net N$10: now also R3.2; no longer R7.1
- net N$11: now also R3.1; no longer R7.2
- net N$2: now also R4.1; no longer R5.2
- net N$3: now also R1.1; no longer R1.2
- net N$4: now also R6.2; no longer R6.1
- net N$5: now also R5.2; no longer R2.2
- net N$6: now also OPTLED2.A, R2.1; no longer LED2.A, R3.1
- net N$7: now also R2.2; no longer R3.2
- net N$8: now also R6.1; no longer R6.2
- net N$9: now also OPTLED1.A, R5.1; no longer LED1.A, R2.1
- net PD0: now also PD0-TXD.2; no longer U2.TXD
- net PD1: now also PD1-RXD.2; no longer U2.RXD
- net PWR: now also ALWAYS-ON.1, C4.1, C5.1, P108.P, P109.P, P110.P, P111.P, P112.P, P211.P, P212.P, P213.P, P214.P, P215.P, P216.P, P217.P, P218.P, P219.P, P220.P, P221.P, P222.P, P223.P, P224.P, P225.P, P226.P, P227.P, P228.P, P229.P, P230.P, P231.P, P232.P, P233.P, P234.P, P235.P, P236.P, P37.P, P38.P, P39.P, P40.P, P41.P, P62.P, P64.P, P71.P, P74.P, P78.P, P79.P, P80.P, P81.P, P82.P, P83.P, P84.P, P85.P, P86.P, P87.P, P88.P, P89.P, P90.P, P91.P, P92.P, P93.P, P94.P, P95.P, P96.P, P97.P, P98.P, P99.P, R1.2, R4.2, R8.2; no longer C7.1, C8.1, POWER-CLOCK.2, POWER-CLOCK.6, R1.1, R4.1, R5.1
- net XTAL1: now also C7.1; no longer C10.1, POWER-CLOCK.5
- net XTAL2: now also C6.1; no longer C9.1, POWER-CLOCK.4
Other:
- note removed: "SMT PARTS?!?! Clear labels? Serial * 1 * 2? ADC .. JTAG .. i2c/twi all the 1's drill holes"
- note removed: "don't use whole pcb? Cut some off? verify connections isp1 in right rotation"
- moved on the sheet: C7, CTSGND, R1, R2, R3, R4, R5
