File: zik80/schem/zik-pcb-sbc-ez80stm100p-r3.sch (EAGLE design)
At the start: 100 parts, among them IC1 7432N, IC2 7404N

Commit message: Finished up zok atmega bob rev1, and zikzak sbc rev3
Parts:
- renumbered S1 to EZ80-RESET, S2 to STM-RESET
Changed lines of the file:
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@@
 <setting verticaltext="up"/>
 </settings>
-<grid distance="0.05" unitdist="inch" unit="inch" style="dots" multiple="1" display="yes" altdistance="0.01" altunitdist="inch" altunit="inch"/>
+<grid distance="0.1" unitdist="inch" unit="inch" style="lines" multiple="1" display="no" altdistance="0.01" altunitdist="inch" altunit="inch"/>
 <layers>
 <layer number="1" name="Top" color="4" fill="1" visible="no" active="no"/>
@@
 <part name="ISPZDI" library="pinhead" deviceset="PINHD-2X3" device=""/>
 <part name="OSCDIL14" library="crystal" deviceset="CRYSTAL_RES-" device="SG51" value="2.5MHz"/>
-<part name="S1" library="SparkFun-Electromechanical" deviceset="SWITCH-MOMENTARY-2" device="PTH"/>
+<part name="EZ80-RESET" library="SparkFun-Electromechanical" deviceset="SWITCH-MOMENTARY-2" device="PTH"/>
 <part name="GND5" library="supply1" deviceset="GND" device=""/>
 <part name="R3" library="rcl" deviceset="R-US_" device="0204/7" value="10K"/>
@@
 <part name="C19" library="rcl" deviceset="C-EU" device="025-025X050" value="2.2uF"/>
 <part name="GND32" library="supply1" deviceset="GND" device=""/>
-<part name="S2" library="SparkFun-Electromechanical" deviceset="SWITCH-MOMENTARY-2" device="PTH"/>
+<part name="STM-RESET" library="SparkFun-Electromechanical" deviceset="SWITCH-MOMENTARY-2" device="PTH"/>
 <part name="GND33" library="supply1" deviceset="GND" device=""/>
 <part name="VGAHDR" library="pinhead" deviceset="PINHD-1X6" device=""/>
@@
 <instance part="ISPZDI" gate="A" x="64.77" y="240.03" rot="MR0"/>
 <instance part="OSCDIL14" gate="A" x="331.47" y="306.07" rot="MR180"/>
-<instance part="S1" gate="G$1" x="43.18" y="73.66" rot="R90"/>
+<instance part="EZ80-RESET" gate="G$1" x="43.18" y="73.66" rot="R90"/>
 <instance part="GND5" gate="1" x="43.18" y="63.5"/>
 <instance part="R3" gate="G$1" x="29.21" y="85.09" rot="R180"/>
@@
 <instance part="C19" gate="G$1" x="690.88" y="228.6"/>
 <instance part="GND32" gate="1" x="690.88" y="217.17"/>
-<instance part="S2" gate="G$1" x="877.57" y="74.93" rot="MR90"/>
+<instance part="STM-RESET" gate="G$1" x="877.57" y="74.93" rot="MR90"/>
 <instance part="GND33" gate="1" x="877.57" y="64.77" rot="MR0"/>
 <instance part="VGAHDR" gate="A" x="937.26" y="353.06"/>
@@
 <net name="GND" class="0">
 <segment>
-<pinref part="S1" gate="G$1" pin="1"/>
+<pinref part="EZ80-RESET" gate="G$1" pin="1"/>
 <wire x1="43.18" y1="68.58" x2="43.18" y2="66.04" width="0.1524" layer="91"/>
 <pinref part="GND5" gate="1" pin="GND"/>
@@
 </segment>
 <segment>
-<pinref part="S2" gate="G$1" pin="1"/>
+<pinref part="STM-RESET" gate="G$1" pin="1"/>
 <wire x1="877.57" y1="69.85" x2="877.57" y2="67.31" width="0.1524" layer="91"/>
 <pinref part="GND33" gate="1" pin="GND"/>
@@
 <net name="ZNRST" class="0">
 <segment>
-<pinref part="S1" gate="G$1" pin="2"/>
+<pinref part="EZ80-RESET" gate="G$1" pin="2"/>
 <wire x1="43.18" y1="78.74" x2="43.18" y2="85.09" width="0.1524" layer="91"/>
 <wire x1="43.18" y1="85.09" x2="72.39" y2="85.09" width="0.1524" layer="91"/>
@@
 <wire x1="873.76" y1="93.98" x2="877.57" y2="93.98" width="0.1524" layer="91"/>
 <label x="880.11" y="93.98" size="1.27" layer="95" rot="MR180" xref="yes"/>
-<pinref part="S2" gate="G$1" pin="2"/>
+<pinref part="STM-RESET" gate="G$1" pin="2"/>
 <wire x1="877.57" y1="93.98" x2="880.11" y2="93.98" width="0.1524" layer="91"/>
 <wire x1="877.57" y1="80.01" x2="877.57" y2="93.98" width="0.1524" layer="91"/>

Commit message: Text description changes to zikzak SBC rev3 pcb schematic, for clarification on component values etc. No pcb actual changes or schem changes.
Parts:
- R18, R24, R28, R30, R32: value (none) -> 2K
- R19, R25, R27, R29, R31: value (none) -> 1K
Other:
- note added: "Diodes are fast low voltage signal diodes; mA is not so important, but fast response time is. Currently trying 1N4148 as widely available and cheap"
- note added: "PA2-3 == serial console PA8-PA12 = serial control in/out PB0-5 = ctrl bus OE WE /CS0-2 /mreq NoMore PB6/PB7 = i2c sda/scl PB8 -> ctrl bus BUSREQ PB9 -> ctrl bus BUSACK PB10/11 == sync PB12 -> vblank -> z80 -> ZPC6 PB13 -> frameready in -> z80 PB14/15 -> BoB (USB?) PC0-5 == RGB PC6-7 = brightness PE - addr bus PD 8..13 .. addr bus PD 14 .. /CS3 PD 15 .. /IOREQ PD 0..7 data bus"
- note added: "ZPD7 -> CLK ZPD6 -> DATA"
- note added: "joy up (z80 tx0) joy down (zip rx0) joy left joy right joy fire2/unused GND ps2 clk ps2 data"
- note removed: "PA2-3 == serial console PA8-PA12 = serial control in/out PB0-5 = ctrl bus OE WE /CS0-2 /mreq NoMore PB6/PB7 = i2c sda/scl PB8 -> ctrl bus BUSREQ PB9 -> ctrl bus BUSACK PB10/11 == sync PB12 -> vblank -> z80 PB13 -> frameready in -> z80 PB14/15 -> BoB (USB?) PC0-5 == RGB PC6-7 = brightness PE - addr bus PD 8..13 .. addr bus PD 14 .. /CS3 PD 15 .. /IOREQ PD 0..7 data bus"
- note removed: "joy up joy down joy left joy right joy fire2/unused GND ps2 clk ps2 data"
Changed lines of the file:
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@@
 <part name="R16" library="rcl" deviceset="R-US_" device="0207/10" value="2K"/>
 <part name="R17" library="rcl" deviceset="R-US_" device="0207/10" value="1K"/>
-<part name="R18" library="rcl" deviceset="R-US_" device="0207/10"/>
-<part name="R19" library="rcl" deviceset="R-US_" device="0207/10"/>
-<part name="R24" library="rcl" deviceset="R-US_" device="0207/10"/>
-<part name="R25" library="rcl" deviceset="R-US_" device="0207/10"/>
+<part name="R18" library="rcl" deviceset="R-US_" device="0207/10" value="2K"/>
+<part name="R19" library="rcl" deviceset="R-US_" device="0207/10" value="1K"/>
+<part name="R24" library="rcl" deviceset="R-US_" device="0207/10" value="2K"/>
+<part name="R25" library="rcl" deviceset="R-US_" device="0207/10" value="1K"/>
 <part name="R26" library="rcl" deviceset="R-US_" device="0207/10" value="10K"/>
 <part name="GND35" library="supply1" deviceset="GND" device=""/>
-<part name="R27" library="rcl" deviceset="R-US_" device="0207/10"/>
-<part name="R28" library="rcl" deviceset="R-US_" device="0207/10"/>
-<part name="R29" library="rcl" deviceset="R-US_" device="0207/10"/>
-<part name="R30" library="rcl" deviceset="R-US_" device="0207/10"/>
-<part name="R31" library="rcl" deviceset="R-US_" device="0207/10"/>
-<part name="R32" library="rcl" deviceset="R-US_" device="0207/10"/>
+<part name="R27" library="rcl" deviceset="R-US_" device="0207/10" value="1K"/>
+<part name="R28" library="rcl" deviceset="R-US_" device="0207/10" value="2K"/>
+<part name="R29" library="rcl" deviceset="R-US_" device="0207/10" value="1K"/>
+<part name="R30" library="rcl" deviceset="R-US_" device="0207/10" value="2K"/>
+<part name="R31" library="rcl" deviceset="R-US_" device="0207/10" value="1K"/>
+<part name="R32" library="rcl" deviceset="R-US_" device="0207/10" value="2K"/>
 <part name="VBATPWRJP" library="pinhead" deviceset="PINHD-1X2" device=""/>
 <part name="C20" library="rcl" deviceset="C-EU" device="025-025X050" value=".1uF"/>
@@
 in that case or serial
 fail.</text>
-<text x="457.2" y="215.9" size="1.778" layer="91" rot="MR0">joy up
-joy down
+<text x="457.2" y="215.9" size="1.778" layer="91" rot="MR0">joy up (z80 tx0)
+joy down (zip rx0)
 joy left
 joy right
@@
 PB9 -&gt; ctrl bus BUSACK
 PB10/11 == sync
-PB12 -&gt; vblank -&gt; z80
+PB12 -&gt; vblank -&gt; z80 -&gt; ZPC6
 PB13 -&gt; frameready in -&gt; z80
 PB14/15 -&gt; BoB (USB?)
@@
 -&gt; also as USB to savd
   using PA11/PA12 as USB</text>
+<text x="238.76" y="266.7" size="2.54" layer="91">ZPD7 -&gt; CLK
+ZPD6 -&gt; DATA</text>
+<text x="929.64" y="280.67" size="2.54" layer="91">Diodes are fast low voltage
+signal diodes; mA is not so
+important, but fast response
+time is.
+Currently trying 1N4148 as
+widely available and cheap</text>
 </plain>
 <instances>
