File: zik80/schem/zik-pcb-sbc-ez80stm100p-r3-shield-r1.brd (EAGLE design)
At the start: 160 x 100 mm, 7 parts

Commit message: Tweaking library some more
Parts:
- VGA1: device VideoConnectors:DB-15-F90+SHIELD-BIG_PADS -> VideoConnectors-skeemod:DB-15-F90+SHIELD-BIG_PADS
- moved VGA1 6.48 mm to (80.0, 10.2)
Changed lines of the file:
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@@
 <element name="U$3" library="skeezix" package="POTWHEEL" value="10K" x="35.56" y="33.02" rot="R90"/>
 <element name="U$4" library="SparkFun-Connectors-skeemod" package="MINI-DIN6" value="MINI-DIN6PTH" x="12.7" y="19.05"/>
-<element name="VGA1" library="VideoConnectors" package="DB-15-F90+SHIELD-BIG_PADS" value="VGA-F90B" x="73.66" y="8.89"/>
 <element name="X2" library="SparkFun-Connectors-skeemod" package="DB9" value="" x="69.85" y="39.37"/>
+<element name="VGA1" library="VideoConnectors-skeemod" package="DB-15-F90+SHIELD-BIG_PADS" value="VGA-F90B" x="80.01" y="10.16"/>
 </elements>
 <signals>

Commit message: Tweaking libraries
Parts:
- X1: device adafruit-musb:4UCONN_20329 -> adafruit-musb-skeemod:4UCONN_20329
- moved X1 3.81 mm to (10.2, 48.3), turned to 0 degrees
Changed lines of the file:
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@@
 <element name="U$1" library="skeezix" package="DCJACKZIK" value="DCJACKZIK" x="5.08" y="26.67"/>
 <element name="U$2" library="skeezix" package="MICROSD10" value="MICROSD10" x="33.02" y="6.35"/>
-<element name="X1" library="adafruit-musb" package="4UCONN_20329" value="" x="10.16" y="44.45" rot="R270"/>
 <element name="U$3" library="skeezix" package="POTWHEEL" value="10K" x="35.56" y="33.02" rot="R90"/>
 <element name="U$4" library="SparkFun-Connectors-skeemod" package="MINI-DIN6" value="MINI-DIN6PTH" x="12.7" y="19.05"/>
 <element name="X2" library="SparkFun-Connectors-skeemod" package="DB9" value="" x="69.85" y="39.37"/>
 <element name="VGA1" library="VideoConnectors-skeemod" package="DB-15-F90+SHIELD-BIG_PADS" value="VGA-F90B" x="80.01" y="10.16"/>
+<element name="X1" library="adafruit-musb-skeemod" package="4UCONN_20329" value="" x="10.16" y="48.26"/>
 </elements>
 <signals>
@@
 <signal name="GND">
 <contactref element="U$1" pad="JACKET"/>
-<contactref element="X1" pad="BASE@1"/>
-<contactref element="X1" pad="BASE@2"/>
+<contactref element="X1" pad="SPRT@4"/>
 <contactref element="X1" pad="GND"/>
 <contactref element="X1" pad="SPRT@1"/>
+<contactref element="X1" pad="BASE@1"/>
 <contactref element="X1" pad="SPRT@2"/>
+<contactref element="X1" pad="BASE@2"/>
 <contactref element="X1" pad="SPRT@3"/>
-<contactref element="X1" pad="SPRT@4"/>
-<wire x1="10.935" y1="43.15" x2="11.06" y2="41.15" width="0" layer="19" extent="1-1"/>
-<wire x1="8.26" y1="40.85" x2="11.06" y2="41.15" width="0" layer="19" extent="1-1"/>
-<wire x1="8.16" y1="43.7" x2="10.935" y2="43.15" width="0" layer="19" extent="1-1"/>
-<wire x1="8.16" y1="45.2" x2="8.16" y2="43.7" width="0" layer="19" extent="1-1"/>
-<wire x1="8.26" y1="48.05" x2="8.16" y2="45.2" width="0" layer="19" extent="1-1"/>
-<wire x1="11.06" y1="47.75" x2="8.26" y2="48.05" width="0" layer="19" extent="1-1"/>
-<wire x1="6.35" y1="32.004" x2="8.26" y2="48.05" width="0" layer="19" extent="1-1"/>
+<wire x1="11.46" y1="49.035" x2="13.46" y2="49.16" width="0" layer="19" extent="1-1"/>
+<wire x1="10.91" y1="46.26" x2="11.46" y2="49.035" width="0" layer="19" extent="1-1"/>
+<wire x1="9.41" y1="46.26" x2="10.91" y2="46.26" width="0" layer="19" extent="1-1"/>
+<wire x1="13.76" y1="45.979" x2="10.91" y2="46.26" width="0" layer="19" extent="1-1"/>
+<wire x1="6.56" y1="45.979" x2="9.41" y2="46.26" width="0" layer="19" extent="1-1"/>
+<wire x1="6.86" y1="49.16" x2="6.56" y2="45.979" width="0" layer="19" extent="1-1"/>
+<wire x1="6.35" y1="32.004" x2="6.56" y2="45.979" width="0" layer="19" extent="1-1"/>
+</signal>
+<signal name="+5V">
+<contactref element="VGA1" pad="9"/>
 </signal>
 <signal name="VBUS">
 <contactref element="X1" pad="VBUS"/>
 </signal>
-<signal name="+5V">
-<contactref element="VGA1" pad="9"/>
-</signal>
 </signals>
