File: zik80/schem/zik-pcb-sbc-ez80stm100p-r3-shield-r1.brd (EAGLE design)
At the start: 149.8 x 100 mm, 46 parts

Commit message: Shield Routing..
Parts:
- turned C1 to 0 degrees
- turned C2 to 180 degrees
Routing:
- net N$8: track 0.00 -> 63.6 mm, vias 0 -> 2
- net N$11: track 0.00 -> 62.0 mm
- net USB5: track 0.00 -> 57.6 mm, vias 0 -> 2
- net N$12: track 0.00 -> 36.8 mm, vias 0 -> 2
- net USB_D+: track 0.00 -> 31.8 mm, vias 0 -> 2
- net DTR: track 0.00 -> 30.5 mm, vias 0 -> 1
- net RTS: track 0.00 -> 29.0 mm
- net USB_D-: track 0.00 -> 27.0 mm, vias 0 -> 2
- net FTDI3: track 0.00 -> 24.6 mm, vias 0 -> 2
- net N$13: track 0.00 -> 22.9 mm
- net DCD: track 0.00 -> 17.3 mm
- net RI: track 0.00 -> 10.4 mm
- net CTS: track 0.00 -> 10.4 mm
- net VCC: track 0.00 -> 7.62 mm
- net PWR5: track 0.00 -> 7.62 mm
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
Commit message: Shield routing
Parts:
- added USBDATA: (no value), pinhead:1X05
- moved C26 21.5 mm to (121.2, 60.3), turned to 90 degrees
- moved C23 6.10 mm to (99.8, 60.6), turned to 90 degrees
- moved C13 3.56 mm to (121.2, 69.6)
- moved R34 1.55 mm to (99.4, 70.2)
Connections:
- net GND: now also USBDATA.5
- net PWR5: now also USBDATA.1
- net SPA10: now also USBDATA.4
- net SPA11: now also USBDATA.2
- net SPA12: now also USBDATA.3
Routing:
- net ZPD4: track 0.00 -> 146.7 mm, vias 0 -> 3
- net ZPD3: track 0.00 -> 128.1 mm, vias 0 -> 3
- net ZPD2: track 0.00 -> 127.9 mm, vias 0 -> 3
- net SV: track 0.00 -> 115.5 mm, vias 0 -> 1
- net SH: track 0.00 -> 107.0 mm, vias 0 -> 1
- net SR: track 0.00 -> 91.4 mm
- net SG: track 0.00 -> 88.8 mm
- net SB: track 0.00 -> 86.1 mm
- net ZPD1: track 0.00 -> 80.6 mm, vias 0 -> 1
- net PWR5: track 7.62 -> 84.8 mm, vias 0 -> 1
- net ZPD0: track 0.00 -> 68.1 mm, vias 0 -> 1
- net USB5: track 57.6 -> 82.6 mm, vias 2 -> 1
- net USB_D-: track 27.0 -> 50.3 mm
- net USB_D+: track 31.8 -> 53.9 mm
- net N$23: track 0.00 -> 14.8 mm
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
Commit message: Shield is routed and checked... ready for boardhouse!
Parts:
- moved R6 5.40 mm to (20.7, 24.0), turned to 270 degrees
- moved R3 2.40 mm to (17.0, 24.1), turned to 270 degrees
- moved TXLED 1.91 mm to (22.9, 11.4)
- moved C3 1.31 mm to (89.5, 65.3)
- moved RXLED 0.77 mm to (15.7, 11.6)
- moved R34 0.38 mm to (99.4, 69.8)
- renumbered U$1 to BARREL
Routing:
- net PWR5: track 84.8 -> 443.5 mm, vias 1 -> 3
- net PWR3: track 7.62 -> 251.5 mm, vias 0 -> 6
- net ZPB3-SCK: track 0.00 -> 206.4 mm, vias 0 -> 5
- net ZPB6-MISO: track 0.00 -> 202.5 mm, vias 0 -> 2
- net ZPB2-SS: track 0.00 -> 201.5 mm, vias 0 -> 7
- net ZPB7-MOSI: track 0.00 -> 189.4 mm, vias 0 -> 3
- net ZPD6_DATA: track 0.00 -> 186.5 mm, vias 0 -> 5
- net ZPD7_CLK: track 0.00 -> 167.7 mm, vias 0 -> 6
- net N$2: track 0.00 -> 160.9 mm, vias 0 -> 4
- net N$23: track 14.8 -> 163.8 mm, vias 0 -> 1
- net N$1: track 0.00 -> 134.7 mm, vias 0 -> 4
- net N$3: track 0.00 -> 75.8 mm
- net ZPD0: track 68.1 -> 140.0 mm, vias 1 -> 3
- net N$6: track 0.00 -> 71.8 mm, vias 0 -> 4
- net ZPC1: track 0.00 -> 61.7 mm
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Other:
- outline, holes or cut-outs redrawn
- board text added: "Zikshield for ZZr3 rev 1 Jeff Mitchell 2016 www.zikzak.ca"
- board text removed: "Zikshield for ZZr3 rev1 Jeff Mitchell 2016"
