File: zik80/schem/zik-pcb-sbc-ez80stm100p-r3-shield-r1.sch (EAGLE design)
At the start: 45 parts, among them IC1 TPS7133QP, U2 FT232RLSSOP

Commit message: Shield pcb rough layout coming together nicely
Connections:
- new net N$14: GPIOC-JOY0.4
- new net N$15: GPIOC-JOY0.5
- new net N$16: GPIOC-JOY0.6
- new net N$17: GPIOC-JOY0.7
- new net N$18: GPIOC-JOY0.8
- new net N$19: PS2KEYB.1
- new net N$20: PS2KEYB.2
- new net N$21: PS2KEYB.3
- new net N$25: PS2KEYB.4
- new net N$26: VGAHDR.1
- new net N$27: VGAHDR.2
- new net N$28: VGAHDR.3
- new net N$29: VGAHDR.4
- new net N$30: VGAHDR.5
- new net N$31: VGAHDR.6
- new net N$5: GPIOC-JOY0.1
- new net N$7: GPIOC-JOY0.2
- new net N$9: GPIOC-JOY0.3
- new net ZPD2: GPIOD-JOY1.3
- new net ZPD3: GPIOD-JOY1.4
- new net ZPD4: GPIOD-JOY1.5
- new net ZPD5: GPIOD-JOY1.6
- net GND: now also U$5.S
- net N$23: now also U$5.R, U$5.T
Other:
- note added: "Schem lib is mislabeled? Should be minus always close to V?"
- note added: "Verify - all pin1 orientations! - ensure cap, resistor sizine/type - printout pcb to printer, eyeball it - PWR v PW5 vs PWR3 vs 5V vs etc .. all powers are hooked right - net review; ensure no +5V and other old net names - uncover reset buttons.. anything else? LEDs? cutout over? - verify USB 5p is correct .. power and D- D+ correct pins - potwheel on right? cmp to r4 - mill in some slots for air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"
- note removed: "Schem lib is mislabeled? Shoudl be minus always close to V?"
- note removed: "Verify - all pin1 orientations! - which jacks can be used, while in middle of pcb - jacks in middle have clearance for SD-pulling, headphone pulling, etc - ensure cap, resistor sizine/type - printout pcb to printer, eyeball it - PWR v PW% vs PWR3 vs 5V vs etc .. all powers are hooked right - net review; ensure no +5V and other old net names - uncover reset buttons.. anything else? LEDs? - verify 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"
- note removed: "todo: headphone jack"
- moved on the sheet: PS2KEYB, U$5
Changed lines of the file:
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@@
 <part name="GND13" library="supply1" deviceset="GND" device=""/>
 <part name="P+4" library="supply1" deviceset="+5V" device=""/>
+<part name="GND14" library="supply1" deviceset="GND" device=""/>
 </parts>
 <sheets>
@@
 <text x="374.65" y="140.97" size="7.62" layer="91">Verify
 - all pin1 orientations!
-- which jacks can be used, while in middle of pcb
-- jacks in middle have clearance for SD-pulling, headphone pulling, etc
 - ensure cap, resistor sizine/type
 - printout pcb to printer, eyeball it
-- PWR v PW% vs PWR3 vs 5V vs etc .. all powers are hooked right
+- PWR v PW5 vs PWR3 vs 5V vs etc .. all powers are hooked right
 - net review; ensure no +5V and other old net names
-- uncover reset buttons.. anything else? LEDs?
+- uncover reset buttons.. anything else? LEDs? cutout over?
 - verify USB 5p is correct .. power and D- D+ correct pins
 - potwheel on right? cmp to r4
 - mill in some slots for air flow? visibility?
-- silkscreen name/branding/rev
-- data USB
+- silkscreen name/branding/rev, pin1s
 - SD, unrouted, DRC, ERC...
 - extra BoB pins? i2c? SPI? all that stuff, bring them up and dont populate?
-- Ensure slot for cart is deep enough for plastic box clearance?
-- case readyness?</text>
+- Ensure slot for cart is deep/wide enough for plastic box clearance?
+- case readyness?
+- remove back milling, hell with it?</text>
 <text x="114.3" y="-119.38" size="2.54" layer="91">Use Vcc12V or +5?
 Decouple Vcc/GND with a cap?</text>
-<text x="116.84" y="-139.7" size="5.08" layer="91">todo: headphone jack</text>
 <text x="12.7" y="-106.68" size="3.81" layer="91">Audio Amp</text>
 <text x="8.89" y="255.27" size="3.81" layer="91">Powering PCB Notes</text>
@@
 OTG_FS_DP</text>
 <text x="-27.94" y="160.02" size="1.778" layer="91">Schem lib is mislabeled?
-Shoudl be minus always
+Should be minus always
 close to V?</text>
 <text x="494.03" y="-17.78" size="1.778" layer="91">Schem lib is mislabeled?
-Shoudl be minus always
+Should be minus always
 close to V?</text>
 </plain>
@@
 <instance part="VGA1" gate="G$1" x="562.61" y="97.79"/>
 <instance part="USBSERPWR" gate="G$1" x="-11.43" y="175.26"/>
-<instance part="U$5" gate="G$1" x="203.2" y="-144.78"/>
+<instance part="U$5" gate="G$1" x="123.19" y="-142.24"/>
 <instance part="GND1" gate="1" x="71.12" y="152.4"/>
 <instance part="GND2" gate="1" x="91.44" y="137.16"/>
@@
 <instance part="VGAHDR" gate="A" x="525.78" y="97.79"/>
 <instance part="BOB-PA" gate="A" x="473.71" y="12.7"/>
-<instance part="PS2KEYB" gate="A" x="438.15" y="100.33"/>
+<instance part="PS2KEYB" gate="A" x="424.18" y="100.33"/>
 <instance part="GNDOUT" gate="A" x="270.51" y="139.7"/>
 <instance part="3V3OUT" gate="A" x="294.64" y="139.7"/>
@@
 <instance part="GND13" gate="1" x="485.14" y="-17.78"/>
 <instance part="P+4" gate="1" x="485.14" y="19.05"/>
+<instance part="GND14" gate="1" x="116.84" y="-146.05"/>
 </instances>
 <busses>
@@
 <wire x1="485.14" y1="-5.08" x2="485.14" y2="-15.24" width="0.1524" layer="91"/>
 <pinref part="GND13" gate="1" pin="GND"/>
+</segment>
+<segment>
+<pinref part="U$5" gate="G$1" pin="S"/>
+<wire x1="123.19" y1="-138.43" x2="116.84" y2="-138.43" width="0.1524" layer="91"/>
+<wire x1="116.84" y1="-138.43" x2="116.84" y2="-143.51" width="0.1524" layer="91"/>
+<pinref part="GND14" gate="1" pin="GND"/>
 </segment>
 </net>
@@
 <segment>
 <pinref part="C25" gate="G$1" pin="-"/>
-<wire x1="111.76" y1="-135.89" x2="115.57" y2="-135.89" width="0.1524" layer="91"/>
+<pinref part="U$5" gate="G$1" pin="R"/>
+<wire x1="111.76" y1="-135.89" x2="116.84" y2="-135.89" width="0.1524" layer="91"/>
+<wire x1="116.84" y1="-135.89" x2="123.19" y2="-135.89" width="0.1524" layer="91"/>
+<wire x1="116.84" y1="-135.89" x2="116.84" y2="-133.35" width="0.1524" layer="91"/>
+<pinref part="U$5" gate="G$1" pin="T"/>
+<wire x1="116.84" y1="-133.35" x2="123.19" y2="-133.35" width="0.1524" layer="91"/>
+<junction x="116.84" y="-135.89"/>
 </segment>
 </net>
@@
 </segment>
 </net>
+<net name="ZPD2" class="0">
+<segment>
+<wire x1="13.97" y1="22.86" x2="22.86" y2="22.86" width="0.1524" layer="91"/>
+<pinref part="GPIOD-JOY1" gate="A" pin="3"/>
+<label x="22.86" y="22.86" size="1.27" layer="95" xref="yes"/>
+</segment>
+</net>
+<net name="ZPD3" class="0">
+<segment>
+<wire x1="13.97" y1="20.32" x2="22.86" y2="20.32" width="0.1524" layer="91"/>
+<pinref part="GPIOD-JOY1" gate="A" pin="4"/>
+<label x="22.86" y="20.32" size="1.27" layer="95" xref="yes"/>
+</segment>
+</net>
+<net name="ZPD4" class="0">
+<segment>
+<wire x1="13.97" y1="17.78" x2="22.86" y2="17.78" width="0.1524" layer="91"/>
+<pinref part="GPIOD-JOY1" gate="A" pin="5"/>
+<label x="22.86" y="17.78" size="1.27" layer="95" xref="yes"/>
+</segment>
+</net>
+<net name="ZPD5" class="0">
+<segment>
+<wire x1="13.97" y1="15.24" x2="22.86" y2="15.24" width="0.1524" layer="91"/>
+<pinref part="GPIOD-JOY1" gate="A" pin="6"/>
+<label x="22.86" y="15.24" size="1.27" layer="95" xref="yes"/>
+</segment>
+</net>
+<net name="N$5" class="0">
+<segment>
+<pinref part="GPIOC-JOY0" gate="A" pin="1"/>
+<wire x1="12.7" y1="78.74" x2="22.86" y2="78.74" width="0.1524" layer="91"/>
+<label x="22.86" y="78.74" size="1.27" layer="95" xref="yes"/>
+</segment>
+</net>
+<net name="N$7" class="0">
+<segment>
+<pinref part="GPIOC-JOY0" gate="A" pin="2"/>
+<wire x1="12.7" y1="76.2" x2="22.86" y2="76.2" width="0.1524" layer="91"/>
+<label x="22.86" y="76.2" size="1.27" layer="95" xref="yes"/>
+</segment>
+</net>
+<net name="N$9" class="0">
+<segment>
+<pinref part="GPIOC-JOY0" gate="A" pin="3"/>
+<wire x1="12.7" y1="73.66" x2="22.86" y2="73.66" width="0.1524" layer="91"/>
+<label x="22.86" y="73.66" size="1.27" layer="95" xref="yes"/>
+</segment>
+</net>
+<net name="N$14" class="0">
+<segment>
+<pinref part="GPIOC-JOY0" gate="A" pin="4"/>
+<wire x1="12.7" y1="71.12" x2="22.86" y2="71.12" width="0.1524" layer="91"/>
+<label x="22.86" y="71.12" size="1.27" layer="95" xref="yes"/>
+</segment>
+</net>
+<net name="N$15" class="0">
+<segment>
+<pinref part="GPIOC-JOY0" gate="A" pin="5"/>
+<wire x1="12.7" y1="68.58" x2="22.86" y2="68.58" width="0.1524" layer="91"/>
+<label x="22.86" y="68.58" size="1.27" layer="95" xref="yes"/>
+</segment>
+</net>
+<net name="N$16" class="0">
+<segment>
+<pinref part="GPIOC-JOY0" gate="A" pin="6"/>
+<wire x1="12.7" y1="66.04" x2="22.86" y2="66.04" width="0.1524" layer="91"/>
+<label x="22.86" y="66.04" size="1.27" layer="95" xref="yes"/>
+</segment>
+</net>
+<net name="N$17" class="0">
+<segment>
+<pinref part="GPIOC-JOY0" gate="A" pin="7"/>
+<wire x1="12.7" y1="63.5" x2="22.86" y2="63.5" width="0.1524" layer="91"/>
+<label x="22.86" y="63.5" size="1.27" layer="95" xref="yes"/>
+</segment>
+</net>
+<net name="N$18" class="0">
+<segment>
+<pinref part="GPIOC-JOY0" gate="A" pin="8"/>
+<wire x1="12.7" y1="60.96" x2="22.86" y2="60.96" width="0.1524" layer="91"/>
+<label x="22.86" y="60.96" size="1.27" layer="95" xref="yes"/>
+</segment>
+</net>
+<net name="N$19" class="0">
+<segment>
+<pinref part="PS2KEYB" gate="A" pin="1"/>
+<wire x1="421.64" y1="105.41" x2="414.02" y2="105.41" width="0.1524" layer="91"/>
+<label x="414.02" y="105.41" size="1.27" layer="95" rot="R180" xref="yes"/>
+</segment>
+</net>
+<net name="N$20" class="0">
+<segment>
+<pinref part="PS2KEYB" gate="A" pin="2"/>
+<wire x1="421.64" y1="102.87" x2="414.02" y2="102.87" width="0.1524" layer="91"/>
+<label x="414.02" y="102.87" size="1.27" layer="95" rot="R180" xref="yes"/>
+</segment>
+</net>
+<net name="N$21" class="0">
+<segment>
+<pinref part="PS2KEYB" gate="A" pin="3"/>
+<wire x1="421.64" y1="100.33" x2="414.02" y2="100.33" width="0.1524" layer="91"/>
+<label x="414.02" y="100.33" size="1.27" layer="95" rot="R180" xref="yes"/>
+</segment>
+</net>
+<net name="N$25" class="0">
+<segment>
+<pinref part="PS2KEYB" gate="A" pin="4"/>
+<wire x1="421.64" y1="97.79" x2="414.02" y2="97.79" width="0.1524" layer="91"/>
+<label x="414.02" y="97.79" size="1.27" layer="95" rot="R180" xref="yes"/>
+</segment>
+</net>
+<net name="N$26" class="0">
+<segment>
+<pinref part="VGAHDR" gate="A" pin="1"/>
+<wire x1="523.24" y1="105.41" x2="514.35" y2="105.41" width="0.1524" layer="91"/>
+<label x="514.35" y="105.41" size="1.27" layer="95" rot="R180" xref="yes"/>
+</segment>
+</net>
+<net name="N$27" class="0">
+<segment>
+<pinref part="VGAHDR" gate="A" pin="2"/>
+<wire x1="523.24" y1="102.87" x2="514.35" y2="102.87" width="0.1524" layer="91"/>
+<label x="514.35" y="102.87" size="1.27" layer="95" rot="R180" xref="yes"/>
+</segment>
+</net>
+<net name="N$28" class="0">
+<segment>
+<pinref part="VGAHDR" gate="A" pin="3"/>
+<wire x1="523.24" y1="100.33" x2="514.35" y2="100.33" width="0.1524" layer="91"/>
+<label x="514.35" y="100.33" size="1.27" layer="95" rot="R180" xref="yes"/>
+</segment>
+</net>
+<net name="N$29" class="0">
+<segment>
+<pinref part="VGAHDR" gate="A" pin="4"/>
+<wire x1="523.24" y1="97.79" x2="514.35" y2="97.79" width="0.1524" layer="91"/>
+<label x="514.35" y="97.79" size="1.27" layer="95" rot="R180" xref="yes"/>
+</segment>
+</net>
+<net name="N$30" class="0">
+<segment>
+<pinref part="VGAHDR" gate="A" pin="5"/>
+<wire x1="523.24" y1="95.25" x2="514.35" y2="95.25" width="0.1524" layer="91"/>
+<label x="514.35" y="95.25" size="1.27" layer="95" rot="R180" xref="yes"/>
+</segment>
+</net>
+<net name="N$31" class="0">
+<segment>
+<pinref part="VGAHDR" gate="A" pin="6"/>
+<wire x1="523.24" y1="92.71" x2="514.35" y2="92.71" width="0.1524" layer="91"/>
+<label x="514.35" y="92.71" size="1.27" layer="95" rot="R180" xref="yes"/>
+</segment>
+</net>

Commit message: Working on the shield and proving jack layouts
Parts:
- removed U$4: MINI-DIN6PTH, SparkFun-Connectors-skeemod:MINI-DIN6PTH
- added PS/2KEYB: MINI-DIN6PTH, SparkFun-Connectors-skeemod:MINI-DIN6PTH
Connections:
- net N$16 renamed ZPC5
- net N$17 renamed ZPC6
- net N$18 renamed ZPC7
- removed net N$14: GPIOC-JOY0.4
- removed net N$15: GPIOC-JOY0.5
- removed net N$19: PS2KEYB.1
- removed net N$20: PS2KEYB.2
- removed net N$21: PS2KEYB.3
- removed net N$25: PS2KEYB.4
- removed net N$5: GPIOC-JOY0.1
- removed net N$7: GPIOC-JOY0.2
- removed net N$9: GPIOC-JOY0.3
- new net ZPC0: GPIOC-JOY0.1, JOY0.5
- new net ZPC1: GPIOC-JOY0.2, JOY0.4
- new net ZPC2: GPIOC-JOY0.3, JOY0.3
- new net ZPC3: GPIOC-JOY0.4, JOY0.2
- new net ZPC4: GPIOC-JOY0.5, JOY0.9
- new net ZPD6_DATA: PS/2KEYB.1, PS2KEYB.4
- new net ZPD7_CLK: PS/2KEYB.5, PS2KEYB.1
- net GND: now also JOY0.7, PS/2KEYB.3, PS2KEYB.2, U$2.SD6
- net PWR3: now also U$2.SD4
- net PWR5: now also JOY0.8, PS/2KEYB.4, PS2KEYB.3
- net ZPB2-SS: now also BOB-PA.5, U$2.SD2
- net ZPB3-SCK: now also BOB-PA.6, U$2.SD5
- net ZPB6-MISO: now also BOB-PA.7, U$2.SD7
- net ZPB7-MOSI: now also BOB-PA.8, U$2.SD3
Other:
- note added: "Checked - ZZ hdr to jack pcb - PS/2 keyb ... ok - SD slot seems okay - JOY0 seems ok"
- note added: "NOTE: This connects STM32 SPI1 to eZ80 SPI .. both are GPIO, so one or both side should be highZ mode!"
- note added: "SPA4 SPI1 NSS SPA5 SPI1 SCK SPA6 SPI1 MISO SPA7 SPI1 MOSI"
- moved on the sheet: BOBGPIOB, JOY0

Commit message: Shield incremental
Connections:
- net GND: now also JOY1.7
- net PWR5: now also JOY1.8
- net ZPD0: now also JOY1.5
- net ZPD1: now also JOY1.4
- net ZPD2: now also JOY1.3
- net ZPD3: now also JOY1.2
- net ZPD4: now also JOY1.9
Other:
- note added: "Checked - ZZ hdr to jack pcb - PS/2 keyb ... ok - SD slot seems okay - JOY0 seems ok - JOY1 seems ok - USB PWR ? - USB Data ? - Barrel ? - headphone? - vga? - thumbwheel?"
- note removed: "Checked - ZZ hdr to jack pcb - PS/2 keyb ... ok - SD slot seems okay - JOY0 seems ok"
- moved on the sheet: JOY1
Changed lines of the file:
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@@
 <part name="P+5" library="supply1" deviceset="+5V" device=""/>
 <part name="GND16" library="SparkFun" deviceset="GND" device=""/>
+<part name="P+6" library="supply1" deviceset="+5V" device=""/>
+<part name="GND17" library="SparkFun" deviceset="GND" device=""/>
 </parts>
 <sheets>
@@
 3V3
 GND</text>
-<text x="5.08" y="8.89" size="1.778" layer="91" rot="MR0">joy up (z80 tx0)
+<text x="63.5" y="8.89" size="1.778" layer="91" rot="MR0">joy up (z80 tx0)
 joy down (zip rx0)
 joy left
@@
 Should be minus always
 close to V?</text>
-<text x="723.9" y="275.59" size="7.62" layer="91">Checked - ZZ hdr to jack pcb
+<text x="762" y="184.15" size="7.62" layer="91">Checked - ZZ hdr to jack pcb
 - PS/2 keyb ... ok
 - SD slot seems okay
-- JOY0 seems ok</text>
+- JOY0 seems ok
+- JOY1 seems ok
+- USB PWR ?
+- USB Data ?
+- Barrel ?
+- headphone?
+- vga?
+- thumbwheel?</text>
 <text x="436.88" y="12.7" size="1.27" layer="91">SPA4 SPI1 NSS
 SPA5 SPI1 SCK
@@
 <instance part="LINEOUT" gate="G$1" x="104.14" y="-87.63" rot="R90"/>
 <instance part="GND42" gate="1" x="101.6" y="-97.79"/>
-<instance part="JOY1" gate="G$1" x="53.34" y="20.32"/>
+<instance part="JOY1" gate="G$1" x="-10.16" y="17.78" rot="MR0"/>
 <instance part="VCC" gate="VCC" x="274.32" y="181.61"/>
 <instance part="GND12" gate="1" x="256.54" y="127"/>
@@
 <instance part="P+5" gate="1" x="-22.86" y="50.8" rot="R180"/>
 <instance part="GND16" gate="1" x="-22.86" y="81.28" rot="R180"/>
+<instance part="P+6" gate="1" x="-21.59" y="0" rot="R180"/>
+<instance part="GND17" gate="1" x="-21.59" y="33.02" rot="R180"/>
 </instances>
 <busses>
@@
 <pinref part="JOY0" gate="G$1" pin="7"/>
 <wire x1="-22.86" y1="69.85" x2="-19.05" y2="69.85" width="0.1524" layer="91"/>
+</segment>
+<segment>
+<pinref part="JOY1" gate="G$1" pin="7"/>
+<wire x1="-17.78" y1="17.78" x2="-21.59" y2="17.78" width="0.1524" layer="91"/>
+<wire x1="-21.59" y1="17.78" x2="-21.59" y2="30.48" width="0.1524" layer="91"/>
+<pinref part="GND17" gate="1" pin="GND"/>
 </segment>
 </net>
@@
 <wire x1="-22.86" y1="67.31" x2="-19.05" y2="67.31" width="0.1524" layer="91"/>
 </segment>
+<segment>
+<pinref part="JOY1" gate="G$1" pin="8"/>
+<wire x1="-17.78" y1="15.24" x2="-21.59" y2="15.24" width="0.1524" layer="91"/>
+<wire x1="-21.59" y1="15.24" x2="-21.59" y2="2.54" width="0.1524" layer="91"/>
+<pinref part="P+6" gate="1" pin="+5V"/>
+</segment>
 </net>
 <net name="ZPD0" class="0">
@@
 <wire x1="13.97" y1="27.94" x2="22.86" y2="27.94" width="0.1524" layer="91"/>
 <label x="22.86" y="27.94" size="1.27" layer="95" xref="yes"/>
+<wire x1="13.97" y1="27.94" x2="6.35" y2="27.94" width="0.1524" layer="91"/>
+<wire x1="6.35" y1="27.94" x2="6.35" y2="12.7" width="0.1524" layer="91"/>
+<pinref part="JOY1" gate="G$1" pin="5"/>
+<wire x1="6.35" y1="12.7" x2="-2.54" y2="12.7" width="0.1524" layer="91"/>
 </segment>
 <segment>
@@
 <wire x1="13.97" y1="25.4" x2="22.86" y2="25.4" width="0.1524" layer="91"/>
 <label x="22.86" y="25.4" size="1.27" layer="95" xref="yes"/>
+<wire x1="13.97" y1="25.4" x2="3.81" y2="25.4" width="0.1524" layer="91"/>
+<wire x1="3.81" y1="25.4" x2="3.81" y2="15.24" width="0.1524" layer="91"/>
+<pinref part="JOY1" gate="G$1" pin="4"/>
+<wire x1="3.81" y1="15.24" x2="-2.54" y2="15.24" width="0.1524" layer="91"/>
 </segment>
 <segment>
@@
 <pinref part="GPIOD-JOY1" gate="A" pin="3"/>
 <label x="22.86" y="22.86" size="1.27" layer="95" xref="yes"/>
+<wire x1="13.97" y1="22.86" x2="1.27" y2="22.86" width="0.1524" layer="91"/>
+<wire x1="1.27" y1="22.86" x2="1.27" y2="17.78" width="0.1524" layer="91"/>
+<pinref part="JOY1" gate="G$1" pin="3"/>
+<wire x1="1.27" y1="17.78" x2="-2.54" y2="17.78" width="0.1524" layer="91"/>
 </segment>
 </net>
@@
 <pinref part="GPIOD-JOY1" gate="A" pin="4"/>
 <label x="22.86" y="20.32" size="1.27" layer="95" xref="yes"/>
+<pinref part="JOY1" gate="G$1" pin="2"/>
+<wire x1="13.97" y1="20.32" x2="-2.54" y2="20.32" width="0.1524" layer="91"/>
 </segment>
 </net>
@@
 <pinref part="GPIOD-JOY1" gate="A" pin="5"/>
 <label x="22.86" y="17.78" size="1.27" layer="95" xref="yes"/>
-</segment>
-</net>
+<wire x1="13.97" y1="17.78" x2="8.89" y2="17.78" width="0.1524" layer="91"/>
+<wire x1="8.89" y1="17.78" x2="8.89" y2="7.62" width="0.1524" layer="91"/>
+<wire x1="8.89" y1="7.62" x2="-19.05" y2="7.62" width="0.1524" layer="91"/>
+<wire x1="-19.05" y1="7.62" x2="-19.05" y2="12.7" width="0.1524" layer="91"/>
+<pinref part="JOY1" gate="G$1" pin="9"/>
+<wire x1="-19.05" y1="12.7" x2="-17.78" y2="12.7" width="0.1524" layer="91"/>
+</segment>
+</net>

Commit message: Shield schem nearly final, just need to lay down traces on pcb
Parts:
- added C13: .1uF, rcl:C-EU025-025X050
- renumbered IC1 to TPS7133, U$5 to HEADPHONE, U2 to FTDI
Connections:
- removed net +5V: U$6.6
- removed net N$26: VGAHDR.1
- removed net N$27: VGAHDR.2
- removed net N$28: VGAHDR.3
- removed net N$29: VGAHDR.4
- removed net N$30: VGAHDR.5
- removed net N$31: VGAHDR.6
- new net SB: VGA1G$1.VGA-B, VGAHDR.6
- new net SG: VGA1G$1.VGA-G, VGAHDR.5
- new net SH: VGA1G$1.VGA-HSYNC, VGAHDR.2
- new net SR: VGA1G$1.VGA-R, VGAHDR.4
- new net SV: VGA1G$1.VGA-VSYNC, VGAHDR.1
- net GND: now also C13.2, SPKR.4, VGA1G$1.GND@0, VGA1G$1.GND@1, VGA1G$1.VGA-B-, VGA1G$1.VGA-G-, VGA1G$1.VGA-R-, VGAHDR.3
- net PWR5: now also C13.1, U$6.6, VGA1G$1.+5V
- net SPA10: now also USBGPU.ID
- net SPA11: now also USBGPU.D-; no longer USBGPU.D+
- net SPA12: now also USBGPU.D+; no longer USBGPU.D-
- net USB_D+: now also USBSERPWR.D+; no longer USBSERPWR.D-
- net USB_D-: now also USBSERPWR.D-; no longer USBSERPWR.D+
Other:
- note added: "Checked - ZZ hdr to jack pcb - PS/2 keyb ... ok - SD slot seems okay - JOY0 seems ok - JOY1 seems ok - USB PWR seem ok - USB Data seem ok - vga seems ok - pot wheel seems ok - Barrel ? unchecked, not relevent; probably right, and can specify polarity on male side eventually - headphone .. should be ok, checked during part build + netlist seems clean, no old floating power +5Vs etc"
- note added: "Legend: p1: vsync: B10 p2: hsync: B11 p3: gnd p4: R p5: G p6: B"
- note added: "NOTE: SD from eZ80 was added later and can conflict with audio. SD activity shouldn't bother audio but possibly audio will fight with SD.."
- note added: "Schem pins not same order as physical jack pin order"
- note added: "Should p9 be + or GND? It _can_ power PNP chip in monitor (or monitor can self power.) If monitor self powers and its gnd on board, short wipes board. If pwr on board and or monitor, will monitor handle PNP chip without SPI on cable? Have to assume yes. So we should either not connect the pin at all, or power it and hope that is correct in all cases."
- note added: "Use Vcc12V or +5?"
- note added: "Verify - ensure cap, resistor sizine/type - printout pcb to printer, eyeball it - SD, unrouted, DRC, ERC... - Ensure slot for cart is deep/wide enough for plastic box clearance? - case readyness?"
- note removed: "Checked - ZZ hdr to jack pcb - PS/2 keyb ... ok - SD slot seems okay - JOY0 seems ok - JOY1 seems ok - USB PWR ? - USB Data ? - Barrel ? - headphone? - vga? - thumbwheel?"
- note removed: "Schem lib is mislabeled? Should be minus always close to V?"
- note removed: "Use Vcc12V or +5? Decouple Vcc/GND with a cap?"
- note removed: "Verify - all pin1 orientations! - ensure cap, resistor sizine/type - printout pcb to printer, eyeball it - PWR v PW5 vs PWR3 vs 5V vs etc .. all powers are hooked right - net review; ensure no +5V and other old net names - uncover reset buttons.. anything else? LEDs? cutout over? - verify USB 5p is correct .. power and D- D+ correct pins - potwheel on right? cmp to r4 - mill in some slots for air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"
- moved on the sheet: VGA1G$1, VGAHDR
