File: zik80/schem/zik-pcb-sbc-ez80stm100p-r3-shield-r1.sch (EAGLE design)
At the start: 46 parts

Commit message: Shield routing
Parts:
- added USBDATA: (no value), pinhead:PINHD-1X5
Connections:
- net GND: now also USBDATA.5
- net PWR5: now also USBDATA.1
- net SPA10: now also USBDATA.4
- net SPA11: now also USBDATA.2
- net SPA12: now also USBDATA.3
Other:
- note added: "V+ D- D+ ID GND"
- moved on the sheet: USBGPU
Changed lines of the file:
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@@
 <part name="C13" library="rcl" deviceset="C-EU" device="025-025X050" value=".1uF"/>
 <part name="GND23" library="supply1" deviceset="GND" device=""/>
+<part name="USBDATA" library="pinhead" deviceset="PINHD-1X5" device=""/>
 </parts>
 <sheets>
@@
 <text x="-25.4" y="161.29" size="1.778" layer="91">Schem pins not same order
 as physical jack pin order</text>
-<text x="491.49" y="-15.24" size="1.778" layer="91">Schem pins not same order
+<text x="544.83" y="-12.7" size="1.778" layer="91">Schem pins not same order
 as physical jack pin order</text>
 <text x="739.14" y="132.08" size="7.62" layer="91">Checked - ZZ hdr to jack pcb
@@
 SD activity shouldn't bother audio
 but possibly audio will fight with SD..</text>
+<text x="505.46" y="13.97" size="1.778" layer="91">V+
+D-
+D+
+ID
+GND</text>
 </plain>
 <instances>
@@
 <instance part="+3V2" gate="G$1" x="281.94" y="124.46" rot="R180"/>
 <instance part="P+3" gate="1" x="308.61" y="124.46" rot="R180"/>
-<instance part="USBGPU" gate="G$1" x="500.38" y="0" rot="MR0"/>
-<instance part="GND13" gate="1" x="485.14" y="-17.78"/>
+<instance part="USBGPU" gate="G$1" x="557.53" y="1.27" rot="MR0"/>
+<instance part="GND13" gate="1" x="490.22" y="-16.51"/>
 <instance part="P+4" gate="1" x="485.14" y="19.05"/>
 <instance part="GND14" gate="1" x="116.84" y="-146.05"/>
@@
 <instance part="C13" gate="G$1" x="146.05" y="-120.65" rot="R90"/>
 <instance part="GND23" gate="1" x="158.75" y="-120.65" rot="R90"/>
+<instance part="USBDATA" gate="A" x="509.27" y="1.27"/>
 </instances>
 <busses>
@@
 </segment>
 <segment>
+<wire x1="490.22" y1="-3.81" x2="490.22" y2="-13.97" width="0.1524" layer="91"/>
+<pinref part="GND13" gate="1" pin="GND"/>
+<wire x1="490.22" y1="-3.81" x2="506.73" y2="-3.81" width="0.1524" layer="91"/>
+<pinref part="USBDATA" gate="A" pin="5"/>
+<wire x1="506.73" y1="-3.81" x2="547.37" y2="-3.81" width="0.1524" layer="91"/>
 <pinref part="USBGPU" gate="G$1" pin="GND"/>
-<wire x1="490.22" y1="-5.08" x2="485.14" y2="-5.08" width="0.1524" layer="91"/>
-<wire x1="485.14" y1="-5.08" x2="485.14" y2="-15.24" width="0.1524" layer="91"/>
-<pinref part="GND13" gate="1" pin="GND"/>
+<junction x="506.73" y="-3.81"/>
 </segment>
 <segment>
@@
 </segment>
 <segment>
+<wire x1="506.73" y1="6.35" x2="485.14" y2="6.35" width="0.1524" layer="91"/>
+<wire x1="485.14" y1="6.35" x2="485.14" y2="16.51" width="0.1524" layer="91"/>
+<pinref part="P+4" gate="1" pin="+5V"/>
 <pinref part="USBGPU" gate="G$1" pin="VBUS"/>
-<wire x1="490.22" y1="5.08" x2="485.14" y2="5.08" width="0.1524" layer="91"/>
-<wire x1="485.14" y1="5.08" x2="485.14" y2="16.51" width="0.1524" layer="91"/>
-<pinref part="P+4" gate="1" pin="+5V"/>
+<wire x1="547.37" y1="6.35" x2="506.73" y2="6.35" width="0.1524" layer="91"/>
+<pinref part="USBDATA" gate="A" pin="1"/>
+<junction x="506.73" y="6.35"/>
 </segment>
 <segment>
@@
 <label x="462.28" y="5.08" size="1.27" layer="95" rot="R180" xref="yes"/>
 <wire x1="471.17" y1="5.08" x2="481.33" y2="5.08" width="0.1524" layer="91"/>
-<wire x1="481.33" y1="5.08" x2="481.33" y2="-2.54" width="0.1524" layer="91"/>
+<wire x1="481.33" y1="5.08" x2="481.33" y2="-1.27" width="0.1524" layer="91"/>
+<wire x1="481.33" y1="-1.27" x2="506.73" y2="-1.27" width="0.1524" layer="91"/>
+<pinref part="USBDATA" gate="A" pin="4"/>
 <pinref part="USBGPU" gate="G$1" pin="ID"/>
-<wire x1="481.33" y1="-2.54" x2="490.22" y2="-2.54" width="0.1524" layer="91"/>
+<wire x1="506.73" y1="-1.27" x2="547.37" y2="-1.27" width="0.1524" layer="91"/>
+<junction x="506.73" y="-1.27"/>
 </segment>
 </net>
@@
 <label x="462.28" y="2.54" size="1.27" layer="95" rot="R180" xref="yes"/>
 <wire x1="471.17" y1="2.54" x2="483.87" y2="2.54" width="0.1524" layer="91"/>
-<wire x1="483.87" y1="2.54" x2="483.87" y2="0" width="0.1524" layer="91"/>
+<wire x1="483.87" y1="2.54" x2="483.87" y2="3.81" width="0.1524" layer="91"/>
+<wire x1="483.87" y1="3.81" x2="506.73" y2="3.81" width="0.1524" layer="91"/>
 <pinref part="USBGPU" gate="G$1" pin="D-"/>
-<wire x1="483.87" y1="0" x2="490.22" y2="0" width="0.1524" layer="91"/>
+<wire x1="506.73" y1="3.81" x2="518.16" y2="3.81" width="0.1524" layer="91"/>
+<wire x1="518.16" y1="3.81" x2="534.67" y2="3.81" width="0.1524" layer="91"/>
+<wire x1="534.67" y1="3.81" x2="534.67" y2="1.27" width="0.1524" layer="91"/>
+<wire x1="534.67" y1="1.27" x2="547.37" y2="1.27" width="0.1524" layer="91"/>
+<pinref part="USBDATA" gate="A" pin="2"/>
+<junction x="506.73" y="3.81"/>
 </segment>
 </net>
@@
 <wire x1="471.17" y1="0" x2="462.28" y2="0" width="0.1524" layer="91"/>
 <label x="462.28" y="0" size="1.27" layer="95" rot="R180" xref="yes"/>
-<wire x1="471.17" y1="0" x2="480.06" y2="0" width="0.1524" layer="91"/>
-<wire x1="480.06" y1="0" x2="480.06" y2="1.27" width="0.1524" layer="91"/>
-<wire x1="480.06" y1="1.27" x2="487.68" y2="1.27" width="0.1524" layer="91"/>
-<wire x1="487.68" y1="1.27" x2="487.68" y2="2.54" width="0.1524" layer="91"/>
+<wire x1="471.17" y1="0" x2="483.87" y2="0" width="0.1524" layer="91"/>
+<wire x1="483.87" y1="0" x2="483.87" y2="1.27" width="0.1524" layer="91"/>
+<wire x1="483.87" y1="1.27" x2="506.73" y2="1.27" width="0.1524" layer="91"/>
 <pinref part="USBGPU" gate="G$1" pin="D+"/>
-<wire x1="487.68" y1="2.54" x2="490.22" y2="2.54" width="0.1524" layer="91"/>
-</segment>
-</net>
+<wire x1="506.73" y1="1.27" x2="519.43" y2="1.27" width="0.1524" layer="91"/>
+<wire x1="519.43" y1="1.27" x2="519.43" y2="2.54" width="0.1524" layer="91"/>
+<wire x1="519.43" y1="2.54" x2="539.75" y2="2.54" width="0.1524" layer="91"/>
+<wire x1="539.75" y1="2.54" x2="539.75" y2="3.81" width="0.1524" layer="91"/>
+<wire x1="539.75" y1="3.81" x2="547.37" y2="3.81" width="0.1524" layer="91"/>
+<pinref part="USBDATA" gate="A" pin="3"/>
+<junction x="506.73" y="1.27"/>
+</segment>
+</net>

Commit message: Shield is routed and checked... ready for boardhouse!
Parts:
- renumbered U$1 to BARREL
Other:
- note added: "- NEVER JUMPER enable these unless barrel power jack or headers are unconnected! - Jumper 5V to feed the board from USB (including TPS) - Jump 3V to enable FTDI to feed board; do not do this if TPS7133 is populated"
- note removed: "- NEVER JUMPER enable these unless barrel power jack or headers are unconnected! - Jumper ONLY ONE of these to use USB for power"
- note removed: "Verify - ensure cap, resistor sizine/type - printout pcb to printer, eyeball it - SD, unrouted, DRC, ERC... - Ensure slot for cart is deep/wide enough for plastic box clearance? - case readyness?"
Changed lines of the file:
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@@
 <setting verticaltext="up"/>
 </settings>
-<grid distance="0.05" unitdist="inch" unit="inch" style="dots" multiple="1" display="yes" altdistance="0.01" altunitdist="inch" altunit="inch"/>
+<grid distance="0.1" unitdist="inch" unit="inch" style="lines" multiple="1" display="no" altdistance="0.01" altunitdist="inch" altunit="inch"/>
 <layers>
 <layer number="1" name="Top" color="4" fill="1" visible="no" active="no"/>
@@
 </classes>
 <parts>
-<part name="U$1" library="skeezix" deviceset="DCJACKZIK" device=""/>
+<part name="BARREL" library="skeezix" deviceset="DCJACKZIK" device=""/>
 <part name="U$2" library="skeezix" deviceset="MICROSD10" device=""/>
 <part name="U$3" library="skeezix" deviceset="POTWHEEL" device="" value="10K"/>
@@
 <text x="77.47" y="218.44" size="1.778" layer="91">USB 5V</text>
 <text x="53.34" y="205.74" size="1.778" layer="91">FTDI OUT 3V3</text>
-<text x="8.89" y="215.9" size="1.778" layer="91">- NEVER JUMPER enable these
+<text x="6.35" y="213.36" size="1.778" layer="91">- NEVER JUMPER enable these
 unless barrel power jack or
 headers are unconnected!
-- Jumper ONLY ONE of these to
-use USB for power</text>
+- Jumper 5V to feed the board from
+USB (including TPS)
+- Jump 3V to enable FTDI to feed board;
+do not do this if TPS7133 is
+populated</text>
 <text x="290.83" y="200.66" size="1.778" layer="91">5V-&gt;3.3V
 regulator</text>
@@
 - GND</text>
 <text x="267.97" y="209.55" size="3.81" layer="91">Power Block</text>
-<text x="374.65" y="140.97" size="7.62" layer="91">Verify
-- ensure cap, resistor sizine/type
-- printout pcb to printer, eyeball it
-- SD, unrouted, DRC, ERC...
-- Ensure slot for cart is deep/wide enough for plastic box clearance?
-- case readyness?</text>
 <text x="118.11" y="-113.03" size="2.54" layer="91">Use Vcc12V or +5?</text>
 <text x="12.7" y="-106.68" size="3.81" layer="91">Audio Amp</text>
@@
 <text x="544.83" y="-12.7" size="1.778" layer="91">Schem pins not same order
 as physical jack pin order</text>
-<text x="739.14" y="132.08" size="7.62" layer="91">Checked - ZZ hdr to jack pcb
+<text x="419.1" y="193.04" size="7.62" layer="91">Checked - ZZ hdr to jack pcb
 - PS/2 keyb ... ok
 - SD slot seems okay
@@
 </plain>
 <instances>
-<instance part="U$1" gate="G$1" x="245.11" y="195.58" rot="R270"/>
+<instance part="BARREL" gate="G$1" x="245.11" y="195.58" rot="R270"/>
 <instance part="U$2" gate="G$1" x="354.33" y="-1.27"/>
 <instance part="U$3" gate="G$1" x="41.91" y="-67.31" rot="R270"/>
@@
 <pinref part="PWRIN" gate="A" pin="4"/>
 <wire x1="247.65" y1="161.29" x2="261.62" y2="161.29" width="0.1524" layer="91"/>
-<pinref part="U$1" gate="G$1" pin="GND"/>
+<pinref part="BARREL" gate="G$1" pin="GND"/>
 <wire x1="261.62" y1="161.29" x2="269.24" y2="161.29" width="0.1524" layer="91"/>
 <label x="269.24" y="161.29" size="1.27" layer="95" xref="yes"/>
@@
 <pinref part="PWRIN" gate="A" pin="2"/>
 <wire x1="250.19" y1="166.37" x2="261.62" y2="166.37" width="0.1524" layer="91"/>
-<pinref part="U$1" gate="G$1" pin="VCC"/>
+<pinref part="BARREL" gate="G$1" pin="VCC"/>
 <wire x1="261.62" y1="166.37" x2="269.24" y2="166.37" width="0.1524" layer="91"/>
 <label x="269.24" y="166.37" size="1.27" layer="95" xref="yes"/>
